File: pcb/boneclamp_rC.brd (EAGLE design)
At the start: 160 x 100 mm, 146 parts, among them IC1 24C, IC2 LM741D, IC3 LM741D, U1 AD8032ARZ-REEL7, U10 ADA4841-2YRZ, U11 ADA4841-2YRZ, U12 ADS8331IBPW, U13 OPA365AIDBVR, U14 REF5040MDREP, U15 OPA365AIDBVR, U16 OPA365AIDBVR, U2 LT1964ES5-5TRMPBF, U3 OPA365AIDBVR, U4 TLV70245DBVT, U5 ADA4841-2YRZ, U6 AD713JRZ-16, U9 ADA4841-2YRZ

Commit message: Minor changes.
Connections:
- net AGND: now also U$42.10
- net VDRIVE: no longer U$42.10
Changed lines of the file:
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@@
 <contactref element="U$12" pad="3"/>
 <contactref element="C11" pad="1"/>
-<wire x1="236.535" y1="67.31" x2="230.185" y2="67.31" width="0" layer="19" extent="1-1"/>
-<wire x1="230.185" y1="45.085" x2="230.185" y2="67.31" width="0" layer="19" extent="1-1"/>
-<wire x1="236.535" y1="45.085" x2="230.185" y2="45.085" width="0" layer="19" extent="1-1"/>
-<wire x1="230.185" y1="22.86" x2="230.185" y2="45.085" width="0" layer="19" extent="1-1"/>
+<contactref element="U$42" pad="10"/>
 <wire x1="236.535" y1="22.86" x2="230.185" y2="22.86" width="0" layer="19" extent="1-1"/>
 <wire x1="228.6762" y1="5.08" x2="230.185" y2="22.86" width="0" layer="19" extent="1-1"/>
@@
 <wire x1="248.6" y1="-2.54" x2="242.885" y2="-2.54" width="0" layer="19" extent="1-1"/>
 <wire x1="244.055" y1="-8.89" x2="242.885" y2="-2.54" width="0" layer="19" extent="1-1"/>
+<wire x1="236.535" y1="45.085" x2="236.535" y2="22.86" width="0" layer="19" extent="1-1"/>
+<wire x1="230.185" y1="45.085" x2="236.535" y2="45.085" width="0" layer="19" extent="1-1"/>
+<wire x1="236.535" y1="67.31" x2="236.535" y2="45.085" width="0" layer="19" extent="1-1"/>
+<wire x1="230.185" y1="67.31" x2="236.535" y2="67.31" width="0" layer="19" extent="1-1"/>
 <wire x1="230.185" y1="-38.735" x2="244.055" y2="-8.89" width="0" layer="19" extent="1-1"/>
 <wire x1="231.2162" y1="-48.895" x2="230.185" y2="-38.735" width="0" layer="19" extent="1-1"/>
@@
 <wire x1="230.185" y1="125.095" x2="230.185" y2="67.31" width="0" layer="19" extent="1-1"/>
 <wire x1="230.185" y1="131.445" x2="230.185" y2="125.095" width="0" layer="19" extent="1-1"/>
-<wire x1="-140.655" y1="-771.525" x2="230.185" y2="131.445" width="0" layer="19" extent="1-1"/>
-<wire x1="-143.09" y1="-765.81" x2="-140.655" y2="-771.525" width="0" layer="19" extent="1-1"/>
-<wire x1="-143.09" y1="-760.73" x2="-143.09" y2="-765.81" width="0" layer="19" extent="1-1"/>
-<wire x1="-143.09" y1="-745.49" x2="-143.09" y2="-760.73" width="0" layer="19" extent="1-1"/>
-<wire x1="-143.09" y1="-740.41" x2="-143.09" y2="-745.49" width="0" layer="19" extent="1-1"/>
-<wire x1="-140.655" y1="-725.835" x2="-143.09" y2="-740.41" width="0" layer="19" extent="1-1"/>
-<wire x1="-139.6238" y1="-716.915" x2="-140.655" y2="-725.835" width="0" layer="19" extent="1-1"/>
-<wire x1="-107.63" y1="-561.34" x2="-139.6238" y2="-716.915" width="0" layer="19" extent="1-1"/>
-<wire x1="-105.73" y1="-554.99" x2="-107.63" y2="-561.34" width="0" layer="19" extent="1-1"/>
-<wire x1="-112.08" y1="-554.99" x2="-105.73" y2="-554.99" width="0" layer="19" extent="1-1"/>
-<wire x1="-118.43" y1="-554.99" x2="-112.08" y2="-554.99" width="0" layer="19" extent="1-1"/>
+<wire x1="50.165" y1="72.39" x2="230.185" y2="67.31" width="0" layer="19" extent="1-1"/>
+<wire x1="25.4" y1="57.658" x2="50.165" y2="72.39" width="0" layer="19" extent="1-1"/>
+<wire x1="20.5994" y1="59.3344" x2="25.4" y2="57.658" width="0" layer="19" extent="1-1"/>
+<wire x1="20.5994" y1="63.246" x2="20.5994" y2="59.3344" width="0" layer="19" extent="1-1"/>
+<wire x1="14.9606" y1="61.2902" x2="20.5994" y2="59.3344" width="0" layer="19" extent="1-1"/>
+<wire x1="9.84" y1="59.69" x2="14.9606" y2="61.2902" width="0" layer="19" extent="1-1"/>
+<wire x1="7.94" y1="63.5" x2="9.84" y2="59.69" width="0" layer="19" extent="1-1"/>
+<wire x1="9.84" y1="67.31" x2="7.94" y2="63.5" width="0" layer="19" extent="1-1"/>
+<wire x1="7.94" y1="55.88" x2="9.84" y2="59.69" width="0" layer="19" extent="1-1"/>
+<wire x1="9.84" y1="52.07" x2="7.94" y2="55.88" width="0" layer="19" extent="1-1"/>
+<wire x1="7.94" y1="48.26" x2="9.84" y2="52.07" width="0" layer="19" extent="1-1"/>
+<wire x1="-83.7692" y1="-167.9702" x2="7.94" y2="48.26" width="0" layer="19" extent="1-1"/>
+<wire x1="-82.97" y1="-177.8" x2="-83.7692" y2="-167.9702" width="0" layer="19" extent="1-1"/>
+<wire x1="-82.97" y1="-184.15" x2="-82.97" y2="-177.8" width="0" layer="19" extent="1-1"/>
+<wire x1="-82.97" y1="-190.5" x2="-82.97" y2="-184.15" width="0" layer="19" extent="1-1"/>
+<wire x1="-83.8454" y1="-220.98" x2="-82.97" y2="-190.5" width="0" layer="19" extent="1-1"/>
+<wire x1="-82.97" y1="-229.87" x2="-83.8454" y2="-220.98" width="0" layer="19" extent="1-1"/>
+<wire x1="-82.97" y1="-236.22" x2="-82.97" y2="-229.87" width="0" layer="19" extent="1-1"/>
+<wire x1="-118.43" y1="-379.095" x2="-82.97" y2="-236.22" width="0" layer="19" extent="1-1"/>
+<wire x1="-118.43" y1="-385.445" x2="-118.43" y2="-379.095" width="0" layer="19" extent="1-1"/>
+<wire x1="-118.43" y1="-391.795" x2="-118.43" y2="-385.445" width="0" layer="19" extent="1-1"/>
+<wire x1="-118.43" y1="-463.55" x2="-118.43" y2="-391.795" width="0" layer="19" extent="1-1"/>
+<wire x1="-118.43" y1="-469.9" x2="-118.43" y2="-463.55" width="0" layer="19" extent="1-1"/>
+<wire x1="-118.43" y1="-481.33" x2="-118.43" y2="-469.9" width="0" layer="19" extent="1-1"/>
+<wire x1="-118.43" y1="-492.76" x2="-118.43" y2="-481.33" width="0" layer="19" extent="1-1"/>
+<wire x1="-120.33" y1="-499.11" x2="-118.43" y2="-492.76" width="0" layer="19" extent="1-1"/>
+<wire x1="-118.43" y1="-505.46" x2="-120.33" y2="-499.11" width="0" layer="19" extent="1-1"/>
+<wire x1="-118.43" y1="-554.99" x2="-118.43" y2="-505.46" width="0" layer="19" extent="1-1"/>
+<wire x1="-112.08" y1="-554.99" x2="-118.43" y2="-554.99" width="0" layer="19" extent="1-1"/>
+<wire x1="-105.73" y1="-554.99" x2="-112.08" y2="-554.99" width="0" layer="19" extent="1-1"/>
 <wire x1="-99.38" y1="-554.99" x2="-105.73" y2="-554.99" width="0" layer="19" extent="1-1"/>
 <wire x1="-100.015" y1="-561.34" x2="-99.38" y2="-554.99" width="0" layer="19" extent="1-1"/>
-<wire x1="-118.43" y1="-505.46" x2="-118.43" y2="-554.99" width="0" layer="19" extent="1-1"/>
-<wire x1="-120.33" y1="-499.11" x2="-118.43" y2="-505.46" width="0" layer="19" extent="1-1"/>
-<wire x1="-118.43" y1="-492.76" x2="-120.33" y2="-499.11" width="0" layer="19" extent="1-1"/>
-<wire x1="-118.43" y1="-481.33" x2="-118.43" y2="-492.76" width="0" layer="19" extent="1-1"/>
-<wire x1="-118.43" y1="-469.9" x2="-118.43" y2="-481.33" width="0" layer="19" extent="1-1"/>
-<wire x1="-118.43" y1="-463.55" x2="-118.43" y2="-469.9" width="0" layer="19" extent="1-1"/>
-<wire x1="-118.43" y1="-391.795" x2="-118.43" y2="-463.55" width="0" layer="19" extent="1-1"/>
-<wire x1="-118.43" y1="-385.445" x2="-118.43" y2="-391.795" width="0" layer="19" extent="1-1"/>
-<wire x1="-118.43" y1="-379.095" x2="-118.43" y2="-385.445" width="0" layer="19" extent="1-1"/>
-<wire x1="-82.97" y1="-236.22" x2="-118.43" y2="-379.095" width="0" layer="19" extent="1-1"/>
-<wire x1="-82.97" y1="-229.87" x2="-82.97" y2="-236.22" width="0" layer="19" extent="1-1"/>
-<wire x1="-83.8454" y1="-220.98" x2="-82.97" y2="-229.87" width="0" layer="19" extent="1-1"/>
-<wire x1="-82.97" y1="-190.5" x2="-83.8454" y2="-220.98" width="0" layer="19" extent="1-1"/>
-<wire x1="-82.97" y1="-184.15" x2="-82.97" y2="-190.5" width="0" layer="19" extent="1-1"/>
-<wire x1="-82.97" y1="-177.8" x2="-82.97" y2="-184.15" width="0" layer="19" extent="1-1"/>
-<wire x1="-83.7692" y1="-167.9702" x2="-82.97" y2="-177.8" width="0" layer="19" extent="1-1"/>
-<wire x1="7.94" y1="48.26" x2="-83.7692" y2="-167.9702" width="0" layer="19" extent="1-1"/>
-<wire x1="9.84" y1="52.07" x2="7.94" y2="48.26" width="0" layer="19" extent="1-1"/>
-<wire x1="7.94" y1="55.88" x2="9.84" y2="52.07" width="0" layer="19" extent="1-1"/>
-<wire x1="9.84" y1="59.69" x2="7.94" y2="55.88" width="0" layer="19" extent="1-1"/>
-<wire x1="7.94" y1="63.5" x2="9.84" y2="59.69" width="0" layer="19" extent="1-1"/>
-<wire x1="9.84" y1="67.31" x2="7.94" y2="63.5" width="0" layer="19" extent="1-1"/>
-<wire x1="14.9606" y1="61.2902" x2="9.84" y2="59.69" width="0" layer="19" extent="1-1"/>
-<wire x1="20.5994" y1="63.246" x2="14.9606" y2="61.2902" width="0" layer="19" extent="1-1"/>
-<wire x1="25.4" y1="57.658" x2="20.5994" y2="63.246" width="0" layer="19" extent="1-1"/>
-<wire x1="50.165" y1="72.39" x2="25.4" y2="57.658" width="0" layer="19" extent="1-1"/>
+<wire x1="-107.63" y1="-561.34" x2="-105.73" y2="-554.99" width="0" layer="19" extent="1-1"/>
+<wire x1="-139.6238" y1="-716.915" x2="-107.63" y2="-561.34" width="0" layer="19" extent="1-1"/>
+<wire x1="-140.655" y1="-725.835" x2="-139.6238" y2="-716.915" width="0" layer="19" extent="1-1"/>
+<wire x1="-143.09" y1="-740.41" x2="-140.655" y2="-725.835" width="0" layer="19" extent="1-1"/>
+<wire x1="-143.09" y1="-745.49" x2="-143.09" y2="-740.41" width="0" layer="19" extent="1-1"/>
+<wire x1="-143.09" y1="-760.73" x2="-143.09" y2="-745.49" width="0" layer="19" extent="1-1"/>
+<wire x1="-143.09" y1="-765.81" x2="-143.09" y2="-760.73" width="0" layer="19" extent="1-1"/>
+<wire x1="-140.655" y1="-771.525" x2="-143.09" y2="-765.81" width="0" layer="19" extent="1-1"/>
 </signal>
 <signal name="DAC_COM">
@@
 <contactref element="R17" pad="2"/>
 <contactref element="R18" pad="2"/>
-<contactref element="U$42" pad="10"/>
 <contactref element="C57" pad="1"/>
 <contactref element="U12" pad="16"/>
@@
 <wire x1="50.165" y1="21.59" x2="-120.33" y2="-372.745" width="0" layer="19" extent="1-1"/>
 <wire x1="52.705" y1="21.59" x2="50.165" y2="21.59" width="0" layer="19" extent="1-1"/>
-<wire x1="20.5994" y1="59.3344" x2="50.165" y2="21.59" width="0" layer="19" extent="1-1"/>
-<wire x1="20.5994" y1="59.9948" x2="20.5994" y2="59.3344" width="0" layer="19" extent="1-1"/>
+<wire x1="20.5994" y1="59.9948" x2="50.165" y2="21.59" width="0" layer="19" extent="1-1"/>
 <wire x1="118.745" y1="21.65" x2="52.705" y2="21.59" width="0" layer="19" extent="1-1"/>
 <wire x1="138.85" y1="24.13" x2="118.745" y2="21.65" width="0" layer="19" extent="1-1"/>

Commit message: Fixed DAC output bias
Biased DAC output, other minor schematic changes
Parts:
- removed D2, D3, D4, D5: 1N4004, diode:DO41-10
- removed IC2, IC3: LM741D, linear:SO08
- removed U11: ADA4841-2YRZ, analog-devices-01:SOIC127P600X175-8N
- added C13, C14, C23, C24, C26, C27, C29, C30, C31, C32, C33, C34, C35, C38, C70, C71, C72, C73: (no value), rcl:C102-043X133
- added R12, R13, R5, R52, R53, R54: 33, rcl:R0603
- added U7, U8: AD8022ARMZ, analog-devices-01:SOP65P490X110-8N
- C25, C28: value 0.1uF -> (none); device rcl:C0805 -> rcl:C102-043X133
- R21, R46: value (none) -> 33; device rcl:PT-10S -> rcl:R0603
- R22, R34, R35, R45: value 1k -> 33; device resistor:0204V -> rcl:R0603
- R31, R38, R43, R44: value 0.1k -> 33; device rcl:R0805 -> rcl:R0603
- R39, R40, R41, R42: value 10k -> 33; device rcl:R0805 -> rcl:R0603
- U10: value ADA4841-2YRZ -> AD8022ARMZ; device analog-devices-01:SOIC127P600X175-8N -> analog-devices-01:SOP65P490X110-8N
- U6: value AD713JRZ-16 -> AD8022ARMZ; device analog-devices-01:SOIC127P1032X265-16N -> analog-devices-01:SOP65P490X110-8N
- moved R22 830.0 mm to (-137.2, 196.8)
- moved C28 816.6 mm to (-137.2, 170.8)
- moved R21 806.5 mm to (-142.2, 196.8)
- moved R34 793.2 mm to (-127.0, 196.8)
- moved R31 638.9 mm to (-132.1, 196.8)
- moved R44 597.6 mm to (-142.2, -1038.2)
- moved R43 592.2 mm to (-142.2, -1033.1)
- moved R42 589.5 mm to (-142.2, -1028.1)
- moved R41 583.8 mm to (-142.2, -1023.0)
- moved R40 578.2 mm to (-142.2, -1017.9)
- moved R39 572.7 mm to (-142.2, -1012.8)
- moved U6 568.9 mm to (-139.7, 152.4)
- moved R38 566.5 mm to (-142.2, -1007.7)
- moved U10 527.5 mm to (-139.7, -959.5)
- moved R46 421.0 mm to (-142.2, -1048.4)
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Connections:
- removed net .5VREF-: IC2.2, R21.1, R34.1, R35.2
- removed net .5VREF-1: C25.1, IC3.2, R46.1
- removed net VBIAS_DOWN: D2.C, D3.C, D4.C, D5.C, IC2.6, R21.2, U6.11, U6.15, U6.2, U6.6
- removed net VBIAS_UP: IC3.6, R31.2, R38.2, R39.1, R39.2, R40.1, R40.2, R41.1, R41.2, R42.1, R42.2, R43.2, R44.2, R46.2, U10.2, U10.6, U11.2, U11.6
- new net N$11: C13.2, R41.1, R43.2, U7.1
- new net N$23: C27.2, R22.1, R34.2, U6.1
- new net N$27: R43.1, R45.2, U10.2
- new net N$30: R35.1, R38.1, R41.2, U7.2
- new net N$31: R44.1, R46.2, U10.6
- new net N$39: R39.1, R40.1, R42.2, U7.6
- new net N$45: C34.2, U10.5
- new net N$46: C33.2, U10.3
- new net N$50: R34.1, R53.2, U8.2
- new net N$52: R52.1, R54.2, U8.6
- new net N$53: R13.1, R21.1, R31.2, U6.6
- new net N$54: R12.1, R22.2, R5.1, U6.2
- new net N$57: C70.2, U8.5
- new net N$58: C38.2, U8.3
- new net _DAC_A_BIASED: R53.1, U8.1
- new net _DAC_BIASED_B: R54.1, U8.7
- new net _DAC_C_BIASED: R45.1, U10.1
- new net _DAC_D_BIASED: R46.1, U10.7
- net ADC_A: no longer U10.3
- net ADC_B: no longer U10.5
- net ADC_C: no longer U11.3
- net ADC_D: no longer U11.5
- net AGND: now also C13.1, C14.1, C23.1, C24.1, C25.1, C26.1, C27.1, C28.1, C29.1, C30.1, C31.1, C32.1, C33.1, C34.1, C35.1, C38.1, C70.1, C71.1, C72.1, C73.1, U6.3, U6.5, U7.3, U7.5
- net GND: no longer C28.2, IC2.3, R45.1, U6.8, U6.9
- net N$10: now also C14.2, R42.1, R44.2, U7.7; no longer IC3.3, R22.1, R45.2
- net N$12: now also C28.2, R31.1, R52.2, U6.7; no longer C28.1, R35.1
- net VBIAS-: now also R21.2, R35.2, R40.2, R5.2
- net VDD: now also C26.2, C32.2, C72.2, C73.2, U6.8, U7.8, U8.8; no longer IC2.7, IC3.7, U11.8, U6.4
- net VREF: no longer R22.2, R34.2
- net VSS: now also C25.2, C31.2, C35.2, C71.2, U6.4, U7.4, U8.4; no longer IC2.4, IC3.4, U11.4, U6.13
- net _ADC_A: no longer R38.1, U10.1
- net _ADC_B: no longer R31.1, U10.7
- net _ADC_C: no longer R43.1, U11.1
- net _ADC_D: no longer R44.1, U11.7
- net _DAC_A: now also C29.2, R12.2; no longer D2.A, U6.14, U6.16
- net _DAC_B: now also C30.2, R13.2; no longer D5.A, U6.1, U6.3
- net _DAC_C: now also C23.2, R38.2; no longer D4.A, U6.5, U6.7
- net _DAC_D: now also C24.2, R39.2; no longer D3.A, U6.10, U6.12
