File: pcb/boneclamp_rC.brd (EAGLE design)
At the start: 160 x 100 mm, 113 parts, among them IC1 24C, U1 AD8032ARZ-REEL7, U12 ADS8331IBPW, U13 OPA365AIDBVR, U14 REF5040MDREP, U15 OPA365AIDBVR, U16 OPA365AIDBVR, U2 OPA365AIDBVR, U3 OPA365AIDBVR, U4 TLV70245DBVT, U5 MAX1735EUK25+T, U6 OPA365AIDBVR, U7 OPA365AIDBVR, U8 OPA365AIDBVR

Commit message: Repackaged passive components.
Shrank all passive components, verified their viability.
Parts:
- C1, C15, C16, C17, C18, C19, C2, C21, C23, C24, C25, C3, C31, C32, C4, C46, C48, C5, C57, C58, C59, C6, C64, C65, C66, C67, C68, C69, C7: device rcl:C0805 -> rcl:C0603
- R1, R17, R18, R2, R3, R4: device rcl:R0805 -> rcl:R0603
- R16, R23: device resistor:R0805 -> rcl:R0603

Commit message: Started implmenenting Amanda's comments.
Connections:
- net VDD renamed +4.5V
- net VSS renamed -4.5V
- net _VREF renamed VREF_PRE
- net _VSS renamed VSS_PRE
- removed net SD: U$12.1
- net AGND: now also U$12.1
Changed lines of the file:
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@@
 <contactref element="U$1" pad="85"/>
 </signal>
-<signal name="VDD">
+<signal name="+4.5V">
 <contactref element="U$42" pad="5"/>
 <contactref element="U$42" pad="5"/>
@@
 <contactref element="C16" pad="2"/>
 <contactref element="SJ4" pad="1"/>
-<contactref element="C9" pad="2"/>
-<contactref element="C8" pad="2"/>
-<contactref element="U4" pad="2"/>
 <contactref element="U$42" pad="4"/>
 <contactref element="U$42" pad="16"/>
@@
 <contactref element="C1" pad="2"/>
 <contactref element="C2" pad="2"/>
-<contactref element="U$12" pad="6"/>
-<contactref element="U$12" pad="3"/>
 <contactref element="C11" pad="1"/>
 <contactref element="U$42" pad="10"/>
 <contactref element="C46" pad="2"/>
-<contactref element="C13" pad="2"/>
 <contactref element="C14" pad="2"/>
-<contactref element="R12" pad="2"/>
-<contactref element="U5" pad="1"/>
 <contactref element="C32" pad="2"/>
 <contactref element="C31" pad="2"/>
@@
 <contactref element="R15" pad="3"/>
 <contactref element="C3" pad="2"/>
+<contactref element="C13" pad="2"/>
+<contactref element="R12" pad="2"/>
+<contactref element="U5" pad="1"/>
+<contactref element="C8" pad="2"/>
+<contactref element="U4" pad="2"/>
+<contactref element="C9" pad="2"/>
+<contactref element="U$12" pad="6"/>
+<contactref element="U$12" pad="3"/>
+<contactref element="U$12" pad="1"/>
 <wire x1="236.435" y1="22.86" x2="230.085" y2="22.86" width="0" layer="19" extent="1-1"/>
 <wire x1="228.6762" y1="5.08" x2="230.085" y2="22.86" width="0" layer="19" extent="1-1"/>
@@
 <wire x1="196.43" y1="-1.27" x2="228.6762" y2="5.08" width="0" layer="19" extent="1-1"/>
 <wire x1="191.35" y1="81.28" x2="230.085" y2="67.31" width="0" layer="19" extent="1-1"/>
-<wire x1="231.2162" y1="-48.895" x2="230.085" y2="-2.54" width="0" layer="19" extent="1-1"/>
+<wire x1="231.2162" y1="-46.355" x2="230.085" y2="-2.54" width="0" layer="19" extent="1-1"/>
+<wire x1="231.2162" y1="-48.895" x2="231.2162" y2="-46.355" width="0" layer="19" extent="1-1"/>
 <wire x1="236.1438" y1="-48.895" x2="231.2162" y2="-48.895" width="0" layer="19" extent="1-1"/>
 <wire x1="227.835" y1="-57.15" x2="231.2162" y2="-48.895" width="0" layer="19" extent="1-1"/>
@@
 <wire x1="25.4" y1="59.182" x2="50.165" y2="74.93" width="0" layer="19" extent="1-1"/>
 </signal>
-<signal name="VSS">
+<signal name="-4.5V">
 <contactref element="C58" pad="1"/>
 <contactref element="U3" pad="2"/>
@@
 <contactref element="U$1" pad="53"/>
 </signal>
-<signal name="_VSS">
+<signal name="VSS_PRE">
 <contactref element="U$12" pad="5"/>
 <contactref element="C11" pad="2"/>
@@
 <wire x1="-42.545" y1="30.48" x2="233.6038" y2="5.08" width="0" layer="19" extent="1-1"/>
 </signal>
-<signal name="_VREF">
-<contactref element="U14" pad="6"/>
-<contactref element="C48" pad="1"/>
-<contactref element="TP9" pad="TP"/>
-<contactref element="U1" pad="3"/>
-<wire x1="189.23" y1="77.47" x2="228.6762" y2="6.35" width="0" layer="19" extent="1-1"/>
-<wire x1="189.65" y1="81.28" x2="189.23" y2="77.47" width="0" layer="19" extent="1-1"/>
-<wire x1="197.4088" y1="137.16" x2="189.65" y2="81.28" width="0" layer="19" extent="1-1"/>
-</signal>
 <signal name="VBIAS+">
 <contactref element="U13" pad="3"/>
@@
 <wire x1="-44.665" y1="-121.285" x2="-36.83" y2="24.765" width="0" layer="19" extent="1-1"/>
 </signal>
-<signal name="SD">
-<contactref element="U$12" pad="1"/>
-</signal>
 <signal name="N$34">
 <contactref element="U$12" pad="4"/>
@@
 <contactref element="U12" pad="13"/>
 </signal>
+<signal name="VREF_PRE">
+<contactref element="U14" pad="6"/>
+<contactref element="C48" pad="1"/>
+<contactref element="TP9" pad="TP"/>
+<contactref element="U1" pad="3"/>
+<wire x1="189.23" y1="77.47" x2="228.6762" y2="6.35" width="0" layer="19" extent="1-1"/>
+<wire x1="189.65" y1="81.28" x2="189.23" y2="77.47" width="0" layer="19" extent="1-1"/>
+<wire x1="197.4088" y1="137.16" x2="189.65" y2="81.28" width="0" layer="19" extent="1-1"/>
+</signal>
 </signals>

Commit message: Took care of most of Amanda's comments. Started using data buses instead of individual nets for the SPI interfaces.
Parts:
- added JP3, JP4: (no value), jumper:JP2
- added JP5: (no value), adafruit:1X03
- added LED1, LED2, LED3, LED4, LED5: (no value), led:CHIPLED_0805
- added R14, R40: 10k, rcl:R0603
- added R24, R34, R35, R36, R39: 2k, rcl:R0603
- added SW1: SPST_TACT, adafruit:EVQ-Q2-A
- added TP11, TP12, TP13: TPB1,27, testpad:B1,27
- added TP14, TP15: TPPAD1-17, testpad:P1-17
Connections:
- net ADC_CNV renamed ADC_SPI4
- net ADC_CS renamed ADC_SPI1
- net ADC_SDO renamed ADC_SPI3
- net DAC_CS renamed DAC_SPI1
- net DAC_SCLK renamed DAC_SPI0
- net N$8 renamed DAC_SPI2
- net _ADC_A renamed ADC_A+
- net _ADC_B renamed ADC_B+
- net _ADC_C renamed ADC_C+
- net _ADC_D renamed ADC_D+
- net _DAC_A renamed DAC_A+
- net _DAC_B renamed DAC_B+
- net _DAC_C renamed DAC_C+
- net _DAC_D renamed DAC_D+
- removed net AGND1: C57.2, U12.14
- removed net DAC_RST: R17.1, U$42.15
- removed net N$37: C55.1, C56.1, C60.1, C61.1, C62.1, C63.1, U12.19, U12.20
- removed net N$7: U$42.8
- removed net PE: C4.2
- new net ADC_SPI0: U12.10
- new net ADC_SPI2: U12.12
- new net DGND1: LED3.C
- new net DGND2: LED4.C
- new net DGND3: LED5.C
- new net GPIO_XX: R34.2, R35.2, R36.2, R39.2
- new net N$11: LED2.A, R34.1
- new net N$20: LED1.A, R24.1
- new net N$23: LED3.A, R35.1
- new net N$25: LED4.A, R36.1
- new net N$26: LED5.A, R39.1
- new net VDD_EXT: R14.1, U$12.1
- new net ~RST: R17.1, R40.1, SW1.A, SW1.A', U$42.15, U12.8
- net +4.5V: now also R24.2, TP12.TP
- net AGND: now also C55.1, C56.1, C60.1, C61.1, C62.1, C63.1, LED1.C, R14.2, TP14.TP, U$42.8, U12.19, U12.20, U12.23; no longer U$12.1
- net DGND: now also C4.2, C57.2, LED2.C, SW1.B, SW1.B', TP15.TP, U12.14
- net VDD_5V: now also JP4.1
- net VDRIVE: now also R40.2
- net VSS_PRE: now also JP3.1, JP3.2, JP4.2, TP13.TP

Commit message: Started renaming test points, etc.
Parts:
- added ADC_A+, ADC_B+, ADC_C+, ADC_D+: TPB1,27, testpad:B1,27
- added EXT_PWR: (no value), led:CHIPLED_0805
- added R41: 2k, rcl:R0603
- renumbered JP2 to A_I/O, JP5 to POW_EXT, LED1 to PWR, SW1 to RESET, TP1 to DAC_D+, TP11 to -4.5V, TP12 to +4.5V, TP13 to VSS_PRE, TP2 to DAC_C+, TP3 to DAC_B+, TP4 to DAC_A+
Connections:
- removed net ADC_COM: A_I/O.2
- removed net DAC_COM: A_I/O.1
- new net N$7: EXT_PWR.A, R41.1
- net AGND: now also A_I/O.1, A_I/O.2, EXT_PWR.C
- net VDD_EXT: now also R41.2

Commit message: More reorganization.
Parts:
- removed LED2, LED3, LED4, LED5: (no value), led:CHIPLED_0805
- removed R35, R36, R39: 2k, rcl:R0603
- C55, C57: value 0.1uF -> 4.7uF
- R34: value 2k -> 10
- moved R34 89.6 mm to (-69.8, -266.1)
- renumbered POW_EXT to PWR_EXT, S2 to ADDRESS, TP10 to VBIAS, TP14 to AGND, TP15 to DGND, TP5 to I2C2_SCLK, TP6 to VDRIVE, TP7 to I2C2_SDA, TP8 to VREF, TP9 to VREF_PRE
Connections:
- net VBIAS+ renamed VBIAS
- removed net DGND1: LED3.C
- removed net DGND2: LED4.C
- removed net DGND3: LED5.C
- removed net GPIO_XX: R34.2, R35.2, R36.2, R39.2
- removed net N$11: LED2.A, R34.1
- removed net N$23: LED3.A, R35.1
- removed net N$25: LED4.A, R36.1
- removed net N$26: LED5.A, R39.1
- new net N$8: R34.2
- new net VSS_EXT: PWR_EXT.3
- net AGND: now also PWR_EXT.2
- net DGND: no longer LED2.C
- net VDD_EXT: now also PWR_EXT.1
- net VREF: now also R34.1

Commit message: Started getting rid of signal tag symbols, take too much room and cause problems with automatic component renumbering.
Connections:
- removed net N$8: R34.2
- net VREF: now also R34.2
Changed lines of the file:
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@@
 <contactref element="U12" pad="20"/>
 <contactref element="C55" pad="1"/>
+<contactref element="A_I/O" pad="1"/>
+<contactref element="A_I/O" pad="2"/>
+<contactref element="EXT_PWR" pad="C"/>
+<contactref element="PWR_EXT" pad="2"/>
 <contactref element="C60" pad="1"/>
 <contactref element="C61" pad="1"/>
@@
 <contactref element="C63" pad="1"/>
 <contactref element="U12" pad="23"/>
-<contactref element="A_I/O" pad="1"/>
-<contactref element="A_I/O" pad="2"/>
-<contactref element="EXT_PWR" pad="C"/>
-<contactref element="PWR_EXT" pad="2"/>
 <wire x1="236.435" y1="22.86" x2="230.085" y2="22.86" width="0" layer="19" extent="1-1"/>
 <wire x1="228.6762" y1="5.08" x2="230.085" y2="22.86" width="0" layer="19" extent="1-1"/>
@@
 <contactref element="VREF" pad="TP"/>
 <contactref element="R34" pad="1"/>
+<contactref element="R34" pad="2"/>
 <wire x1="228.6762" y1="7.62" x2="228.6762" y2="8.89" width="0" layer="19" extent="1-1"/>
 <wire x1="190.715" y1="68.58" x2="228.6762" y2="8.89" width="0" layer="19" extent="1-1"/>
@@
 <wire x1="-42.965" y1="-115.57" x2="-44.665" y2="-115.57" width="0" layer="19" extent="1-1"/>
 <wire x1="-45.085" y1="-127" x2="-44.665" y2="-115.57" width="0" layer="19" extent="1-1"/>
-<wire x1="-70.7" y1="-266.065" x2="-45.085" y2="-127" width="0" layer="19" extent="1-1"/>
+<wire x1="-69" y1="-266.065" x2="-45.085" y2="-127" width="0" layer="19" extent="1-1"/>
+<wire x1="-70.7" y1="-266.065" x2="-69" y2="-266.065" width="0" layer="19" extent="1-1"/>
 </signal>
 <signal name="~RST">
@@
 <wire x1="-68.58" y1="-257.59" x2="-70.7" y2="-260.985" width="0" layer="19" extent="1-1"/>
 </signal>
-<signal name="N$8">
-<contactref element="R34" pad="2"/>
-</signal>
 </signals>

Commit message: Renumbered all components.
Parts:
- removed C56: 22uF, rcl:C0603
- removed C57: 4.7uF, rcl:C0603
- removed C58, C59, C64, C65, C66, C67, C68, C69: 0.1uF, rcl:C0603
- removed C60, C61, C62, C63: 1nF, rcl:C0603
- removed IC1: 24C, on-semiconductor-01:SO-08
- removed R47, R49: 20k, rcl:R0603
- removed R48, R50: 10k, rcl:R0603
- added C26: 10uF, rcl:C0805
- added C27, C28, C41, C42, C45: 0.1uF, rcl:C0603
- added C29, C30: (no value), rcl:C0603
- added C33: 47uF, rcl:C1206
- added C34, C35, C36, C37: 1uF, rcl:C0603
- added C44: 10uF, rcl:C0603
- added R35: 10k, rcl:R0603
- added R36: (no value), boneclamp:M84-TRIMMER
- added R39: 4.75k, rcl:R0603
- added R42: 5.6k, rcl:R0603
- added U9: OPA365AIDBVR, ti-extended:SOT95P280X145-5N
- C1: value 10uF -> 0.1uF
- C11, C12: value 47uF -> 1nF; device rcl:C1206 -> rcl:C0603
- C13, C14: value 1uF -> 1nF
- C15: value (none) -> 22uF
- C16, C17, C18: value (none) -> 0.1uF
- C20: value 10uF -> 0.1uF; device rcl:C0805 -> rcl:C0603
- C25, C31: value 0.1uF -> (none)
- C32: value 0.1uF -> 47uF; device rcl:C0603 -> rcl:C1206
- C8: value 1uF -> 0.1uF
- C9: value 1uF -> 4.7uF
- JP1: device jumper:JP1 -> jumper:JP2
- JP3: device jumper:JP2 -> jumper:JP1
- R1, R2: value (none) -> 20k
- R10: value 5.6k -> 20
- R11, R13: value 10k -> 20
- R12: value 100k -> 20
- R14: value 10k -> 10
- R15: value (none) -> 10k; device boneclamp:M84-TRIMMER -> rcl:R0603
- R19, R29: value 20k -> 10k
- R23: value 10k -> (none)
- R24: value 2k -> 10k
- R25: value 20 -> 10k
- R26, R27, R28: value 20 -> (none)
- R3, R4: value (none) -> 10k
- R30: value 10k -> 100k
- R31: value 10k -> 260k
- R32, R33: value 10k -> 2k
- R34: value 10 -> 10k
- R37, R38: value 10k -> 4.75k
- R41: value 2k -> 5.6k
- R5: value 260k -> 20k
- R6: value 5.6k -> 20k
- R7, R8, R9: value 4.75k -> 10k
- U1: value AD8032ARZ-REEL7 -> OPA365AIDBVR; device analog-devices-02:SOIC127P600X175-8N -> ti-extended:SOT95P280X145-5N
- U12: value ADS8331IBPW -> MAX1735EUK25+T; device ti-extended:SOP65P640X120-24N -> Maxim_By_element14_Batch_1:SOT95P280X145-5N
- U13: value OPA365AIDBVR -> TLV70245DBVT; device ti-extended:SOT95P280X145-5N -> ti-extended:SOT95P280X110-5N
- U15: value OPA365AIDBVR -> AD8032ARZ-REEL7; device ti-extended:SOT95P280X145-5N -> analog-devices-02:SOIC127P600X175-8N
- U16: value OPA365AIDBVR -> 24C; device ti-extended:SOT95P280X145-5N -> on-semiconductor-01:SO-08
- U4: value TLV70245DBVT -> OPA365AIDBVR; device ti-extended:SOT95P280X110-5N -> ti-extended:SOT95P280X145-5N
- U5: value MAX1735EUK25+T -> ADS8331IBPW; device Maxim_By_element14_Batch_1:SOT95P280X145-5N -> ti-extended:SOP65P640X120-24N
- moved R24 412.1 mm to (274.3, 94.6)
- moved U12 371.9 mm to (-2.54, 165.1)
- moved U5 371.9 mm to (265.4, -92.7)
- moved R29 358.8 mm to (-52.7, -137.8)
- moved R41 334.7 mm to (139.7, 0.00)
- moved C3 319.2 mm to (235.6, 45.1)
- moved C24 316.3 mm to (274.3, 101.0)
- moved C21 312.8 mm to (-36.2, 62.9)
- moved C19 311.8 mm to (-36.2, 85.1)
- moved R18 311.3 mm to (-36.8, 79.4)
- moved R17 311.2 mm to (-36.8, 101.6)
- moved C32 310.3 mm to (229.2, -63.5)
- moved C20 307.4 mm to (-29.8, 62.9)
- moved R33 297.7 mm to (-69.8, -261.0)
- moved R9 296.3 mm to (-59.1, -214.6)
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- renumbered C46 to C43, C47 to C40, C48 to C38, C55 to C10, JP4 to JP2, SJ4 to SJ1, U$1 to BB1, U$12 to U11, U$42 to U10
Connections:
- net +4.5V: now also C1.1, C16.1, C18.1, C22.1, C26.1, C27.1, C3.1, C37.1, C41.1, C5.1, C7.1, R32.2, U1.5, U15.8, U5.17, U9.5; no longer C19.1, C2.1, C23.1, C25.1, C32.1, C59.1, C6.1, C65.1, C67.1, C69.1, C9.1, R24.2, U1.8, U12.17, U15.5, U16.5
- net -4.5V: now also C17.1, C19.1, C2.1, C21.1, C23.1, C35.1, C4.1, C6.1, C8.1, R31.2, U1.2, U12.5, U4.2, U9.2; no longer C14.1, C24.1, C31.1, C5.1, C58.1, C64.1, C66.1, C68.1, C7.1, R5.2, U13.2, U15.2, U16.2, U5.5
- net ADC_A: now also R1.2; no longer R19.2
- net ADC_A+: now also R10.2, R3.1, U1.1; no longer R20.1, R25.2, U3.1
- net ADC_B: now also R5.2; no longer R29.2
- net ADC_B+: now also R11.2, R7.1, U3.1; no longer R26.2, R30.1, U13.1
- net ADC_C: now also R2.2; no longer R47.2
- net ADC_C+: now also R12.2, R4.1, U2.1; no longer R27.2, R48.1, U15.1
- net ADC_D: now also R6.2; no longer R49.2
- net ADC_D+: now also R13.2, R8.1, U4.1; no longer R28.2, R50.1, U16.1
- net ADC_SPI0: now also U5.10; no longer U12.10
- net ADC_SPI1: now also U5.11; no longer U12.11
- net ADC_SPI2: now also U5.12; no longer U12.12
- net ADC_SPI3: now also U5.13; no longer U12.13
- net ADC_SPI4: now also U5.15; no longer U12.15
- net AGND: now also C12.1, C13.1, C14.1, C15.1, C22.2, C26.2, C27.2, C29.2, C30.2, C33.1, C34.2, C35.2, C36.2, C37.2, C4.2, C41.2, C42.2, C44.2, R23.1, R26.1, R27.1, R29.2, R30.2, R36.3, U12.1, U13.2, U15.4, U5.19, U5.20, U5.23; no longer C13.2, C14.2, C31.2, C32.2, C56.1, C58.2, C59.2, C60.1, C61.1, C62.1, C63.1, C64.2, C65.2, C66.2, C67.2, C68.2, C69.2, C9.2, R12.2, R14.2, R15.3, R2.1, R3.1, R4.1, U1.4, U12.19, U12.20, U12.23, U4.2, U5.1
- net DAC_A: now also R17.1, U6.1; no longer R38.1, U2.1
- net DAC_A+: now also C31.1, R28.2, U6.3; no longer C15.1, R1.2, U2.3
- net DAC_B: now also R21.1, U8.1; no longer R31.1, U7.1
- net DAC_B+: now also C30.1, R27.2, U8.3; no longer C16.1, R2.2, U7.3
- net DAC_C: now also R18.1, U7.1; no longer R21.1, U6.1
- net DAC_C+: now also C29.1, R26.2, U7.3; no longer C17.1, R3.2, U6.3
- net DAC_D: now also R22.1, U9.1; no longer R33.1, U8.1
- net DAC_D+: now also C25.1, R23.2, U9.3; no longer C18.1, R4.2, U8.3
- net DAC_LDAC: now also R25.1; no longer R18.1
- net DGND: now also C28.2, C45.2, C9.2, U16.4, U5.14; no longer C22.2, C4.2, C57.2, IC1.4, U12.14
- net I2C2_SCL: now also R41.1, U16.6; no longer IC1.6, R10.1
- net I2C2_SDA: now also R42.1, U16.5; no longer IC1.5, R6.1
- net N$1: now also R16.1, R18.2, U7.4; no longer R13.1, R21.2, U6.4
- net N$10: now also R20.1, R22.2, U9.4; no longer R32.1, R33.2, U8.4
- net N$13: now also R2.1, R4.2, U2.4; no longer R47.1, R48.2, U15.4
- net N$14: now also R37.1, U16.1; no longer IC1.1, R7.1
- net N$15: now also R6.1, R8.2, U4.4; no longer R49.1, R50.2, U16.4
- net N$17: now also C31.2, R28.1; no longer C15.2, R1.1
- net N$18: now also R38.1, U16.2; no longer IC1.2, R8.1
- net N$19: now also R39.1, U16.3; no longer IC1.3, R9.1
- net N$2: now also R19.1, R21.2, U8.4; no longer R22.1, R31.2, U7.4
- net N$20: now also R32.1; no longer R24.1
- net N$21: now also JP3.2, U16.7; no longer IC1.7, JP1.2
- net N$22: now also JP3.1, R40.1; no longer JP1.1, R11.1
- net N$24: now also U5.21, U5.22; no longer U12.21, U12.22
- net N$3: now also R1.1, R3.2, U1.4; no longer R19.1, R20.2, U3.4
- net N$33: now also C32.1; no longer C12.1
- net N$34: now also C32.2; no longer C12.2
- net N$39: now also R15.1, R17.2, U6.4; no longer R37.1, R38.2, U2.4
- net N$4: now also C44.1, R36.2, U15.5; no longer C1.1, R15.2, U1.5
- net N$40: now also C11.2, R10.1, U5.24; no longer C60.2, R25.1, U12.24
- net N$41: now also C12.2, R11.1, U5.1; no longer C61.2, R26.1, U12.1
- net N$42: now also C13.2, R12.1, U5.2; no longer C62.2, R27.1, U12.2
- net N$43: now also C14.2, R13.1, U5.3; no longer C63.2, R28.1, U12.3
- net N$5: now also R30.1, R31.1, U12.4; no longer R12.1, R5.1, U5.4
- net N$6: now also R5.1, R7.2, U3.4; no longer R29.1, R30.2, U13.4
- net N$7: now also R33.1; no longer R41.1
- net N$9: now also R35.2, U15.6, U15.7; no longer R23.2, U1.6, U1.7
- net VBIAS: now also R35.1, U1.3, U2.3, U4.3; no longer R23.1, U13.3, U15.3, U16.3
- net VDD_5V: now also C36.1, U13.1, U13.3; no longer C8.1, U4.1, U4.3
- net VDD_EXT: now also R29.1, R33.2; no longer R14.1, R41.2
- net VDRIVE: now also C28.1, C45.1, C9.1, R24.2, R25.2, R37.2, R38.2, R39.2, R41.2, R42.2, U16.8, U5.16; no longer C22.1, C4.1, C57.1, IC1.8, R10.2, R11.2, R17.2, R18.2, R6.2, R7.2, R8.2, U12.16
- net VREF: now also C15.2, C24.1, C42.1, R14.1, R14.2, R15.2, R19.2, R20.2, R36.1, U15.1, U15.2, U5.18; no longer C21.1, C3.1, C56.2, R13.2, R15.1, R16.1, R22.2, R32.2, R37.2, U1.1, U1.2, U12.18
- net VREF_PRE: now also U15.3; no longer U1.3
- net VSS_PRE: now also C33.2, C34.1, JP1.1, JP1.2, U12.2, U12.3; no longer C11.2, C13.1, JP3.1, JP3.2, U5.2, U5.3
- net ~RST: now also R24.1, R9.1, U5.8; no longer R17.1, R40.1, U12.8
