File: pcb/boneclamp_rC.brd (EAGLE design)
At the start: 54.6 x 86.4 mm, 133 parts, among them U1 OPA365AIDBVR, U10 AD5686, U11 LM2663, U12 MAX1735, U13 TLV70245, U14 REF5040MDREP, U15 AD8032ARZ-REEL7, U16 24C, U2 OPA365AIDBVR, U3 OPA365AIDBVR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

Commit message: Minor changes.
Routing:
- net VSS_PRE: track 22.1 -> 21.2 mm
Changed lines of the file:
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@@
 <element name="C41" library="rcl" package="C0603" value="0.1uF" x="229.235" y="-2.54"/>
 <element name="U11" library="ti-extended" package="SOIC127P600X175-8N" value="LM2663" x="44.323" y="8.255" smashed="yes" rot="R270">
-<attribute name="NAME" x="44.3484" y="7.8232" size="0.8128" layer="25" ratio="10" rot="SR0"/>
+<attribute name="NAME" x="42.2402" y="9.2456" size="0.8128" layer="25" ratio="10" rot="SR270"/>
 <attribute name="VALUE" x="40.6146" y="10.9474" size="1.016" layer="27" ratio="10" rot="SR270"/>
 </element>
@@
 <contactref element="BB1" pad="48"/>
 <wire x1="43.688" y1="5.7912" x2="43.688" y2="7.366" width="0.8128" layer="1"/>
-<via x="43.688" y="9.144" extent="1-16" drill="0.5"/>
-<via x="43.688" y="7.366" extent="1-16" drill="0.5"/>
+<via x="43.688" y="9.144" extent="1-16" drill="0.381"/>
+<via x="43.688" y="7.366" extent="1-16" drill="0.381"/>
 <wire x1="43.688" y1="9.144" x2="43.688" y2="10.7188" width="0.8128" layer="1"/>
-<via x="45.085" y="4.2164" extent="1-16" drill="0.5" shape="octagon"/>
-<via x="46.7106" y="2.7686" extent="1-16" drill="0.5" shape="octagon"/>
+<via x="45.085" y="4.2164" extent="1-16" drill="0.381"/>
+<via x="46.7106" y="2.7686" extent="1-16" drill="0.381"/>
 <wire x1="45.085" y1="4.2164" x2="45.085" y2="2.794" width="0.6096" layer="1"/>
 <wire x1="45.085" y1="2.794" x2="46.736" y2="2.794" width="0.6096" layer="1"/>
@@
 <vertex x="14.351" y="27.94"/>
 </polygon>
-<wire x1="275.17" y1="120.015" x2="191.45" y2="49.53" width="0" layer="19" extent="1-1"/>
-<wire x1="32.258" y1="26.162" x2="191.45" y2="49.53" width="0" layer="19" extent="1-1"/>
-<wire x1="1.8" y1="13.045" x2="10.9" y2="13.045" width="0" layer="19" extent="1-1"/>
-<wire x1="10.248" y1="21.844" x2="10.9" y2="13.045" width="0" layer="19" extent="1-1"/>
-<wire x1="14.157" y1="27.94" x2="10.248" y2="21.844" width="0" layer="19" extent="1-1"/>
-<wire x1="9.906" y1="38.1" x2="14.157" y2="27.94" width="0" layer="19" extent="1-1"/>
-<wire x1="22.225" y1="41.402" x2="9.906" y2="38.1" width="0" layer="19" extent="1-1"/>
 <wire x1="10.9" y1="13.045" x2="12.609" y2="13.045" width="1.4224" layer="1"/>
 <wire x1="12.609" y1="13.045" x2="13.97" y2="11.684" width="1.4224" layer="1"/>
 <wire x1="13.97" y1="11.684" x2="13.97" y2="8.255" width="1.4224" layer="1"/>
+<wire x1="275.17" y1="120.015" x2="191.45" y2="49.53" width="0" layer="19" extent="1-1"/>
+<wire x1="32.258" y1="26.162" x2="191.45" y2="49.53" width="0" layer="19" extent="1-1"/>
+<wire x1="10.248" y1="21.844" x2="10.9" y2="13.045" width="0" layer="19" extent="1-1"/>
+<wire x1="14.157" y1="27.94" x2="10.248" y2="21.844" width="0" layer="19" extent="1-1"/>
+<wire x1="1.8" y1="13.045" x2="10.9" y2="13.045" width="0" layer="19" extent="1-1"/>
+<wire x1="9.906" y1="38.1" x2="14.157" y2="27.94" width="0" layer="19" extent="1-1"/>
+<wire x1="22.225" y1="41.402" x2="9.906" y2="38.1" width="0" layer="19" extent="1-1"/>
 </signal>
 <signal name="-4.5V">
@@
 <wire x1="17.438" y1="24.638" x2="16.256" y2="24.638" width="0" layer="19" extent="1-1"/>
 <wire x1="17.438" y1="22.098" x2="16.256" y2="22.098" width="0" layer="19" extent="1-1"/>
-<wire x1="8.957" y1="24.13" x2="9.398" y2="30.099" width="0" layer="19" extent="1-1"/>
-<wire x1="8.548" y1="21.844" x2="8.957" y2="24.13" width="0" layer="19" extent="1-1"/>
-<wire x1="13.677" y1="21.844" x2="8.957" y2="24.13" width="0" layer="19" extent="1-1"/>
+<wire x1="13.677" y1="21.844" x2="16.256" y2="22.098" width="0" layer="19" extent="1-1"/>
+<wire x1="8.548" y1="21.844" x2="13.677" y2="21.844" width="0" layer="19" extent="1-1"/>
+<wire x1="8.957" y1="24.13" x2="8.548" y2="21.844" width="0" layer="19" extent="1-1"/>
 <wire x1="11.2014" y1="38.1" x2="10.58" y2="30.099" width="0" layer="19" extent="1-1"/>
 <wire x1="-5.7912" y1="38.5826" x2="11.2014" y2="38.1" width="0" layer="19" extent="1-1"/>
@@
 <vertex x="42.672" y="5.334"/>
 </polygon>
-<wire x1="40.386" y1="8.382" x2="42.418" y2="6.35" width="1.4224" layer="1"/>
-<wire x1="42.418" y1="6.35" x2="42.418" y2="5.7912" width="1.4224" layer="1"/>
-<wire x1="40.386" y1="8.382" x2="40.386" y2="18.690790625" width="1.4224" layer="1"/>
+<wire x1="40.386" y1="7.493" x2="40.386" y2="18.690790625" width="1.4224" layer="1"/>
 <wire x1="40.386" y1="18.690790625" x2="40.31160625" y2="18.87039375" width="1.4224" layer="1" curve="44.999502"/>
 <wire x1="42.288" y1="2.667" x2="38.967209375" y2="2.667" width="0.4064" layer="1"/>
@@
 <wire x1="40.31160625" y1="18.87039375" x2="38.862" y2="20.32" width="1.4224" layer="1"/>
 <wire x1="38.862" y1="20.32" x2="38.862" y2="22.86" width="1.4224" layer="1"/>
+<wire x1="40.386" y1="7.493" x2="41.529" y2="6.35" width="1.4224" layer="1"/>
+<polygon width="0" layer="1" thermals="no">
+<vertex x="42.545" y="5.334"/>
+<vertex x="41.529" y="5.334"/>
+<vertex x="41.021" y="5.842"/>
+<vertex x="41.021" y="5.969"/>
+<vertex x="41.91" y="6.858"/>
+<vertex x="42.799" y="6.858"/>
+<vertex x="42.799" y="5.334"/>
+</polygon>
 </signal>
 <signal name="ADC_D">
@@
 <wire x1="11.8618" y1="43.942" x2="273.47" y2="94.615" width="0" layer="19" extent="1-1"/>
 <wire x1="-3.2004" y1="38.5826" x2="11.8618" y2="43.942" width="0" layer="19" extent="1-1"/>
-<wire x1="11.977" y1="21.844" x2="-3.2004" y2="38.5826" width="0" layer="19" extent="1-1"/>
+<wire x1="11.977" y1="21.844" x2="11.8618" y2="43.942" width="0" layer="19" extent="1-1"/>
 <wire x1="10.9" y1="8.545" x2="11.977" y2="21.844" width="0" layer="19" extent="1-1"/>
 <wire x1="1.8" y1="8.545" x2="10.9" y2="8.545" width="0" layer="19" extent="1-1"/>
