File: board/puggleboard_1v0.brd (EAGLE design)
At the start: 54.6 x 86.4 mm, 136 parts, among them U1 OPA365AIDBVR, U10 AD5686, U11 LM2663, U12 MAX1735, U13 TLV70245, U14 REF5040, U15 AD8032, U16 24C, U2 OPA365AIDBVR, U3 OPA365AIDBVR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

Commit message: Created a bill of materials for both boards.
Parts:
- U1, U2, U3, U4, U6, U8, U9: value OPA365AIDBVR -> OPA365
Changed lines of the file:
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@@
 <attribute name="VALUE" x="10.0838" y="46.0248" size="0.6096" layer="27" font="vector" ratio="10" rot="SR0"/>
 </element>
-<element name="U1" library="ti-extended" package="SOT95P280X145-5N" value="OPA365AIDBVR" x="10.414" y="62.484" smashed="yes" rot="R180">
+<element name="U1" library="ti-extended" package="SOT95P280X145-5N" value="OPA365" x="10.414" y="62.484" smashed="yes" rot="R180">
 <attribute name="PACKAGE" value="SOT-23-5" x="10.414" y="62.484" size="1.778" layer="27" rot="R180" display="off"/>
 <attribute name="OC_NEWARK" value="03M9400" x="10.414" y="62.484" size="1.778" layer="27" rot="R180" display="off"/>
@@
 <attribute name="VALUE" x="40.767" y="63.5" size="0.6096" layer="27" font="vector" rot="R90"/>
 </element>
-<element name="U3" library="ti-extended" package="SOT95P280X145-5N" value="OPA365AIDBVR" x="20.701" y="62.484" smashed="yes" rot="R180">
+<element name="U3" library="ti-extended" package="SOT95P280X145-5N" value="OPA365" x="20.701" y="62.484" smashed="yes" rot="R180">
 <attribute name="PACKAGE" value="SOT-23-5" x="20.701" y="62.484" size="1.778" layer="27" rot="R180" display="off"/>
 <attribute name="OC_NEWARK" value="03M9400" x="20.701" y="62.484" size="1.778" layer="27" rot="R180" display="off"/>
@@
 <attribute name="VALUE" x="19.05" y="59.055" size="0.6096" layer="27" font="vector" rot="R180"/>
 </element>
-<element name="U2" library="ti-extended" package="SOT95P280X145-5N" value="OPA365AIDBVR" x="30.988" y="71.755" smashed="yes" rot="R180">
+<element name="U2" library="ti-extended" package="SOT95P280X145-5N" value="OPA365" x="30.988" y="71.755" smashed="yes" rot="R180">
 <attribute name="PACKAGE" value="SOT-23-5" x="30.988" y="71.755" size="1.778" layer="27" rot="R180" display="off"/>
 <attribute name="OC_NEWARK" value="03M9400" x="30.988" y="71.755" size="1.778" layer="27" rot="R180" display="off"/>
@@
 <attribute name="VALUE" x="29.083" y="68.326" size="0.6096" layer="27" font="vector" rot="R180"/>
 </element>
-<element name="U4" library="ti-extended" package="SOT95P280X145-5N" value="OPA365AIDBVR" x="41.275" y="71.755" smashed="yes" rot="R180">
+<element name="U4" library="ti-extended" package="SOT95P280X145-5N" value="OPA365" x="41.275" y="71.755" smashed="yes" rot="R180">
 <attribute name="PACKAGE" value="SOT-23-5" x="41.275" y="71.755" size="1.778" layer="27" rot="R180" display="off"/>
 <attribute name="OC_NEWARK" value="03M9400" x="41.275" y="71.755" size="1.778" layer="27" rot="R180" display="off"/>
@@
 <attribute name="VALUE" x="31.623" y="43.18" size="0.6096" layer="27" font="vector"/>
 </element>
-<element name="U6" library="ti-extended" package="SOT95P280X145-5N" value="OPA365AIDBVR" x="10.414" y="71.755" smashed="yes" rot="R180">
+<element name="U6" library="ti-extended" package="SOT95P280X145-5N" value="OPA365" x="10.414" y="71.755" smashed="yes" rot="R180">
 <attribute name="PACKAGE" value="SOT-23-5" x="10.414" y="71.755" size="1.778" layer="27" rot="R180" display="off"/>
 <attribute name="OC_NEWARK" value="03M9400" x="10.414" y="71.755" size="1.778" layer="27" rot="R180" display="off"/>
@@
 <attribute name="NAME" x="32.004" y="77.089" size="0.6096" layer="25" font="vector"/>
 </element>
-<element name="U8" library="ti-extended" package="SOT95P280X145-5N" value="OPA365AIDBVR" x="20.701" y="71.755" smashed="yes" rot="R180">
+<element name="U8" library="ti-extended" package="SOT95P280X145-5N" value="OPA365" x="20.701" y="71.755" smashed="yes" rot="R180">
 <attribute name="PACKAGE" value="SOT-23-5" x="20.701" y="71.755" size="1.778" layer="27" rot="R180" display="off"/>
 <attribute name="OC_NEWARK" value="03M9400" x="20.701" y="71.755" size="1.778" layer="27" rot="R180" display="off"/>
@@
 <attribute name="VALUE" x="18.796" y="68.326" size="0.6096" layer="27" font="vector" rot="R180"/>
 </element>
-<element name="U9" library="ti-extended" package="SOT95P280X145-5N" value="OPA365AIDBVR" x="41.275" y="81.026" smashed="yes" rot="R180">
+<element name="U9" library="ti-extended" package="SOT95P280X145-5N" value="OPA365" x="41.275" y="81.026" smashed="yes" rot="R180">
 <attribute name="PACKAGE" value="SOT-23-5" x="41.275" y="81.026" size="1.778" layer="27" rot="R180" display="off"/>
 <attribute name="OC_NEWARK" value="03M9400" x="41.275" y="81.026" size="1.778" layer="27" rot="R180" display="off"/>
