File: board/puggleboard_1v0.sch (EAGLE design)
At the start: 136 parts, among them U1 OPA365AIDBVR, U10 AD5686, U11 LM2663, U12 MAX1735, U13 TLV70245, U14 REF5040, U15 AD8032, U16 24C, U2 OPA365AIDBVR, U3 OPA365AIDBVR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

Commit message: Created a bill of materials for both boards.
Parts:
- U1, U2, U3, U4, U6, U8, U9: value OPA365AIDBVR -> OPA365
Changed lines of the file:
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@@
 <part name="R25" library="rcl" deviceset="R-US_" device="R0603" value="10k"/>
 <part name="U5" library="ti-extended" deviceset="ADS8331IBPW" device="" value="ADS8331"/>
-<part name="U1" library="ti-extended" deviceset="OPA365AIDBVR" device=""/>
+<part name="U1" library="ti-extended" deviceset="OPA365AIDBVR" device="" value="OPA365"/>
 <part name="R1" library="rcl" deviceset="R-US_" device="R0603" value="20k"/>
 <part name="R3" library="rcl" deviceset="R-US_" device="R0603" value="10k"/>
@@
 <part name="C14" library="rcl" deviceset="C-EU" device="C0603" value="1nF"/>
 <part name="SUPPLY18" library="supply2" deviceset="AGND" device=""/>
-<part name="U3" library="ti-extended" deviceset="OPA365AIDBVR" device=""/>
+<part name="U3" library="ti-extended" deviceset="OPA365AIDBVR" device="" value="OPA365"/>
 <part name="R5" library="rcl" deviceset="R-US_" device="R0603" value="20k"/>
 <part name="R7" library="rcl" deviceset="R-US_" device="R0603" value="10k"/>
@@
 <part name="C5" library="rcl" deviceset="C-EU" device="C0603" value="0.1uF"/>
 <part name="SUPPLY19" library="supply2" deviceset="AGND" device=""/>
-<part name="U2" library="ti-extended" deviceset="OPA365AIDBVR" device=""/>
+<part name="U2" library="ti-extended" deviceset="OPA365AIDBVR" device="" value="OPA365"/>
 <part name="R2" library="rcl" deviceset="R-US_" device="R0603" value="20k"/>
 <part name="R4" library="rcl" deviceset="R-US_" device="R0603" value="10k"/>
@@
 <part name="C3" library="rcl" deviceset="C-EU" device="C0603" value="0.1uF"/>
 <part name="SUPPLY35" library="supply2" deviceset="AGND" device=""/>
-<part name="U4" library="ti-extended" deviceset="OPA365AIDBVR" device=""/>
+<part name="U4" library="ti-extended" deviceset="OPA365AIDBVR" device="" value="OPA365"/>
 <part name="R6" library="rcl" deviceset="R-US_" device="R0603" value="20k"/>
 <part name="R8" library="rcl" deviceset="R-US_" device="R0603" value="10k"/>
@@
 <part name="R30" library="rcl" deviceset="R-US_" device="R0603" value="100k"/>
 <part name="R31" library="rcl" deviceset="R-US_" device="R0603" value="261k"/>
-<part name="U6" library="ti-extended" deviceset="OPA365AIDBVR" device=""/>
+<part name="U6" library="ti-extended" deviceset="OPA365AIDBVR" device="" value="OPA365"/>
 <part name="R15" library="rcl" deviceset="R-US_" device="R0603" value="10k"/>
 <part name="R17" library="rcl" deviceset="R-US_" device="R0603" value="10k"/>
@@
 <part name="C18" library="rcl" deviceset="C-EU" device="C0603" value="0.1uF"/>
 <part name="SUPPLY9" library="supply2" deviceset="AGND" device=""/>
-<part name="U8" library="ti-extended" deviceset="OPA365AIDBVR" device=""/>
+<part name="U8" library="ti-extended" deviceset="OPA365AIDBVR" device="" value="OPA365"/>
 <part name="R19" library="rcl" deviceset="R-US_" device="R0603" value="10k"/>
 <part name="R21" library="rcl" deviceset="R-US_" device="R0603" value="10k"/>
@@
 <part name="C20" library="rcl" deviceset="C-EU" device="C0603" value="0.1uF"/>
 <part name="SUPPLY20" library="supply2" deviceset="AGND" device=""/>
-<part name="U9" library="ti-extended" deviceset="OPA365AIDBVR" device=""/>
+<part name="U9" library="ti-extended" deviceset="OPA365AIDBVR" device="" value="OPA365"/>
 <part name="R20" library="rcl" deviceset="R-US_" device="R0603" value="10k"/>
 <part name="R22" library="rcl" deviceset="R-US_" device="R0603" value="10k"/>
