File: board/PuggleBoard.sch (EAGLE design)
At the start: 136 parts, among them U1 OPA365, U10 AD5686, U11 LM2663, U12 MAX1735, U13 TLV70245, U14 REF5040, U15 AD8032, U16 24C, U2 OPA365, U3 OPA365, U4 OPA365, U5 ADS8331, U6 OPA365, U7 OPA365, U8 OPA365, U9 OPA365

Commit message: Started to revise board.
Parts:
- removed J_V+, J_V-: (no value), jumper:JP2E
- added JP_POW: (no value), jumper:JP3Q
- added R43: 10k, rcl:R-US_R0603
- C34: value 1uF -> 10uF
- R10, R11, R12, R13: value 20 -> 100
Connections:
- removed net ADC_SPI0: BB1.GPIO2_12, U5.FS/~CS
- removed net ADC_SPI3: BB1.GPIO2_13, U5.~CONVST
- removed net N$23: C34.1, J_V-.2, U12.IN, U12.~SHDN
- new net SPI0: U5.FS/~CS
- new net SPI1: U10.SYNC*
- new net SPI2: U10.SCLK, U5.SCLK
- new net SPI3: U10.SDIN, U5.SDI
- new net SPI4: U10.SDO, U5.SDO
- new net SPI5: U5.~CONVST
- new net VDD_COM: C36.1, JP_POW.4, U13.EN, U13.IN
- new net VSS_COM: C34.1, JP_POW.3, U12.IN, U12.~SHDN
- net ADC_SPI1: no longer U5.SDI
- net ADC_SPI2: no longer U5.SDO
- net DAC_SPI0: no longer U10.SYNC*
- net DAC_SPI1: no longer U10.SDIN
- net DAC_SPI2: no longer U10.SDO
- net DGND: no longer U10.RSTSEL
- net N$11: now also R43.1, U10.RSTSEL; no longer C36.1, J_V+.2, U13.EN, U13.IN
- net SPI_CLK: no longer U10.SCLK, U5.SCLK
- net VDD_5V: now also JP_POW.2; no longer J_V+.3
- net VDD_EXT: now also JP_POW.6; no longer J_V+.1
- net VDRIVE: now also R43.2
- net VSS_EXT: now also JP_POW.5; no longer J_V-.3
- net VSS_PRE: now also JP_POW.1; no longer J_V-.1
Other:
- note added: "SPI BUS MAPPING 1. ADC_CS (SPI0) 2. DAC_CS (SPI1) 3. SCLK (SPI2) 4. MOSI (SPI3) 5. MISO (SPI4) 6. CONVST (SPI5)"
- note removed: "ADC_SPI MAPPING 1. ADC_CS (ADC_SPI0) 2. ADC_SDI (ADC_SPI1) 3. ADC_SDO (ADC_SPI2) 4. ADC_CNV (ADC_SPI3)"
- note removed: "DAC_SPI MAPPING 1. DAC_CS (DAC_SPI0) 2. DAC_SDI (DAC_SPI1) 3. DAC_SDO (DAC_SPI2)"
- note removed: "DAC_SPI MAPPING 1. DAC_SCLK (DAC_SPI0) 2. DAC_CS (DAC_SPI1) 3. DAC_SDI (DAC_SPI2) 4. DAC_SDO (DAC_SPI3)"
- note removed: "GLOBAL 1. SPI_CLK (CLK FOR BOTH DAC AND ADC)"
- moved on the sheet: PWR_EXT, R24, R25, RESET

Commit message: Working through v1.0 fixes.
Parts:
- removed ADDRESS: SWS003, smd-special:SWS003
- removed C16, C17, C18, C19, C20, C21, C22, C23, C7, C8: 0.1uF, rcl:C-EUC0603
- removed J_~W: (no value), jumper:JP1E
- removed R21, R22: 10k, rcl:R-US_R0603
- removed U2, U3, U4, U6, U7, U8, U9: OPA365, ti-extended:OPA365AIDBVR
- added C47, C48: 1uF, rcl:C-EUC0603
- added EEPROM_WP: TPB1,27, testpad:TPB1,27
- added R44, R45: 680, rcl:R-US_R0603
- added S1: SWS002, smd-special:SWS002
- added U17: OPA4209AIPWMOD, ti-extended:OPA4209AIPWMOD
- C5, C6: value 0.1uF -> 1uF
- R1, R2, R5: value 20k -> 680
- R15, R16, R17, R18, R19, R20, R7: value 10k -> 680
- R3, R4, R8: value 10k -> 340
- R6: value 20k -> 340
- U1: value OPA365 -> OPA4209AIPWMOD; device ti-extended:OPA365AIDBVR -> ti-extended:OPA4209AIPWMOD
Connections:
- removed net N$1: R16.1, R18.2, U7.-IN
- removed net N$10: R20.1, R22.2, U9.-IN
- removed net N$13: R2.1, R4.2, U2.-IN
- removed net N$15: R6.1, R8.2, U4.-IN
- removed net N$2: R19.1, R21.2, U8.-IN
- removed net N$21: J_~W.2, U16.WP
- removed net N$3: R1.1, R3.2, U1.-IN
- removed net N$39: R15.1, R17.2, U6.-IN
- removed net N$6: R5.1, R7.2, U3.-IN
- new net ADC_-IN_A: R1.1, R3.2, U17.-IN_A
- new net ADC_-IN_B: R2.1, R4.2, U17.-IN_B
- new net ADC_-IN_C: R5.1, R6.2, U17.-IN_C
- new net ADC_-IN_D: R7.1, R8.2, U17.-IN_D
- new net DAC_+IN_A: U1.+IN_A
- new net DAC_+IN_B: U1.+IN_B
- new net DAC_+IN_C: U1.+IN_C
- new net DAC_+IN_D: U1.+IN_D
- new net DAC_-IN_A: R44.1, R45.2, U1.-IN_A
- new net DAC_-IN_B: R15.1, R16.2, U1.-IN_B
- new net DAC_-IN_C: R17.1, R18.2, U1.-IN_C
- new net DAC_-IN_D: R19.1, R20.2, U1.-IN_D
- net +4.5V: now also C4.1, C48.1, C6.1, U17.V+; no longer C16.1, C18.1, C20.1, C22.1, C3.1, C5.1, C7.1, U2.V+, U3.V+, U4.V+, U6.V+, U7.V+, U8.V+, U9.V+
- net -4.5V: now also C3.1, C47.1, C5.1, U17.V-; no longer C17.1, C19.1, C21.1, C23.1, C4.1, C6.1, C8.1, U2.V-, U3.V-, U4.V-, U6.V-, U7.V-, U8.V-, U9.V-
- net ADC_A+: now also U17.OUT_A; no longer U1.VOUT
- net ADC_B: now also R2.2; no longer R5.2
- net ADC_B+: now also R4.1, U17.OUT_B; no longer R7.1, U3.VOUT
- net ADC_C: now also R5.2; no longer R2.2
- net ADC_C+: now also R6.1, U17.OUT_C; no longer R4.1, U2.VOUT
- net ADC_D: now also R7.2; no longer R6.2
- net ADC_D+: now also U17.OUT_D; no longer U4.VOUT
- net AGND: now also C47.2, C48.2; no longer C16.2, C17.2, C18.2, C19.2, C20.2, C21.2, C22.2, C23.2, C7.2, C8.2
- net DAC_A: now also R45.1, U1.OUT_A; no longer R17.1, U6.VOUT
- net DAC_A+: no longer U6.+IN
- net DAC_B: now also R16.1, U1.OUT_B; no longer R21.1, U8.VOUT
- net DAC_B+: no longer U8.+IN
- net DAC_C: now also U1.OUT_C; no longer U7.VOUT
- net DAC_C+: no longer U7.+IN
- net DAC_D: now also R20.1, U1.OUT_D; no longer R22.1, U9.VOUT
- net DAC_D+: no longer U9.+IN
- net DGND: now also S1.1, S1.2; no longer ADDRESS.1, ADDRESS.2, ADDRESS.3
- net N$14: now also S1.3; no longer ADDRESS.6
- net N$18: now also S1.4; no longer ADDRESS.5
- net N$19: no longer ADDRESS.4
- net N$22: now also EEPROM_WP.TP, U16.WP; no longer J_~W.1
- net VBIAS: now also U17.+IN_A, U17.+IN_B, U17.+IN_C, U17.+IN_D; no longer U1.+IN, U2.+IN, U3.+IN, U4.+IN
- net VREF: now also R17.2, R44.2; no longer R16.2, R20.2
Other:
- moved on the sheet: ADC_A+, ADC_B+, ADC_C+, ADC_D+, C1, C2, R1, R15, R16, R17, R18, R19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

Commit message: More board mods and design notes.
Connections:
- new net PGND: C33.1, R29.2, U11.GND, U11.LV
- net AGND: now also C9.2, U5.DGND; no longer C33.1, R29.2, U11.GND, U11.LV
- net DGND: no longer C9.2, U5.DGND
Changed lines of the file:
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@@
 <setting verticaltext="up"/>
 </settings>
-<grid distance="0.1" unitdist="inch" unit="inch" style="lines" multiple="1" display="yes" altdistance="0.01" altunitdist="inch" altunit="inch"/>
+<grid distance="0.1" unitdist="inch" unit="inch" style="lines" multiple="1" display="no" altdistance="0.01" altunitdist="inch" altunit="inch"/>
 <layers>
 <layer number="1" name="Top" color="4" fill="1" visible="no" active="no"/>
@@
 <part name="C15" library="rcl" deviceset="C-EU" device="C0603" value="22uF"/>
 <part name="C9" library="rcl" deviceset="C-EU" device="C0805" value="4.7uF"/>
-<part name="DGND5" library="supply2" deviceset="PE" device="" value="DGND"/>
 <part name="SUPPLY11" library="supply2" deviceset="AGND" device=""/>
 <part name="C2" library="rcl" deviceset="C-EU" device="C0603" value="0.1uF"/>
@@
 <part name="U11" library="ti-extended" deviceset="LM2663" device=""/>
 <part name="C33" library="rcl" deviceset="C-US" device="C1206" value="47uF"/>
-<part name="SUPPLY37" library="supply2" deviceset="AGND" device=""/>
 <part name="C32" library="rcl" deviceset="C-US" device="C1206" value="47uF"/>
 <part name="C43" library="rcl" deviceset="C-EU" device="C0603" value="0.1uF"/>
@@
 <part name="SUPPLY25" library="supply2" deviceset="AGND" device=""/>
 <part name="SUPPLY26" library="supply2" deviceset="AGND" device=""/>
-<part name="SUPPLY27" library="supply2" deviceset="AGND" device=""/>
-<part name="SUPPLY28" library="supply2" deviceset="AGND" device=""/>
-<part name="SUPPLY30" library="supply2" deviceset="AGND" device=""/>
 <part name="R29" library="rcl" deviceset="R-US_" device="R0603" value="10k"/>
 <part name="-4.5V" library="testpad" deviceset="TP" device="B1,27"/>
@@
 <part name="S1" library="smd-special" deviceset="SWS002" device=""/>
 <part name="EEPROM_WP" library="testpad" deviceset="TP" device="B1,27"/>
+<part name="SUPPLY9" library="supply2" deviceset="AGND" device=""/>
+<part name="GND1" library="supply1" deviceset="GND" device="" value="PGND"/>
+<part name="GND2" library="supply1" deviceset="GND" device="" value="PGND"/>
+<part name="GND3" library="supply1" deviceset="GND" device="" value="PGND"/>
+<part name="GND4" library="supply1" deviceset="GND" device="" value="PGND"/>
 </parts>
 <sheets>
@@
 <instance part="C15" gate="G$1" x="38.1" y="48.26" rot="R180"/>
 <instance part="C9" gate="G$1" x="-116.84" y="81.28"/>
-<instance part="DGND5" gate="PE" x="-116.84" y="22.86"/>
 <instance part="SUPPLY11" gate="G$1" x="-88.9" y="30.48"/>
 <instance part="C2" gate="G$1" x="12.7" y="147.32"/>
@@
 <instance part="R7" gate="G$1" x="-48.26" y="149.86" rot="R180"/>
 <instance part="R8" gate="G$1" x="-38.1" y="139.7" rot="R90"/>
+<instance part="SUPPLY9" gate="G$1" x="-116.84" y="17.78"/>
 </instances>
 <busses>
@@
 <junction x="2.54" y="180.34"/>
 <pinref part="U17" gate="A" pin="V+"/>
-</segment>
-</net>
-<net name="DGND" class="0">
-<segment>
-<pinref part="C9" gate="G$1" pin="2"/>
-<wire x1="-116.84" y1="76.2" x2="-116.84" y2="25.4" width="0.1524" layer="91"/>
-<pinref part="U5" gate="A" pin="DGND"/>
-<wire x1="50.8" y1="33.02" x2="10.16" y2="33.02" width="0.1524" layer="91"/>
-<wire x1="10.16" y1="33.02" x2="10.16" y2="25.4" width="0.1524" layer="91"/>
-<wire x1="10.16" y1="25.4" x2="-116.84" y2="25.4" width="0.1524" layer="91"/>
-<pinref part="DGND5" gate="PE" pin="PE"/>
-<junction x="-116.84" y="25.4"/>
 </segment>
 </net>
@@
 <pinref part="C47" gate="G$1" pin="2"/>
 <wire x1="2.54" y1="139.7" x2="2.54" y2="142.24" width="0.1524" layer="91"/>
+</segment>
+<segment>
+<pinref part="C9" gate="G$1" pin="2"/>
+<wire x1="-116.84" y1="76.2" x2="-116.84" y2="25.4" width="0.1524" layer="91"/>
+<pinref part="U5" gate="A" pin="DGND"/>
+<wire x1="50.8" y1="33.02" x2="10.16" y2="33.02" width="0.1524" layer="91"/>
+<wire x1="10.16" y1="33.02" x2="10.16" y2="25.4" width="0.1524" layer="91"/>
+<wire x1="10.16" y1="25.4" x2="-116.84" y2="25.4" width="0.1524" layer="91"/>
+<pinref part="SUPPLY9" gate="G$1" pin="AGND"/>
+<wire x1="-116.84" y1="20.32" x2="-116.84" y2="25.4" width="0.1524" layer="91"/>
+<junction x="-116.84" y="25.4"/>
 </segment>
 </net>
@@
 <instance part="U11" gate="G$1" x="2.54" y="35.56"/>
 <instance part="C33" gate="G$1" x="40.64" y="15.24" rot="R180"/>
-<instance part="SUPPLY37" gate="G$1" x="40.64" y="5.08"/>
 <instance part="C32" gate="G$1" x="-35.56" y="35.56"/>
 <instance part="U12" gate="A" x="2.54" y="-12.7"/>
@@
 <instance part="SUPPLY25" gate="G$1" x="-17.78" y="-30.48"/>
 <instance part="SUPPLY26" gate="G$1" x="30.48" y="-86.36"/>
-<instance part="SUPPLY27" gate="G$1" x="27.94" y="5.08"/>
-<instance part="SUPPLY28" gate="G$1" x="-25.4" y="5.08"/>
-<instance part="SUPPLY30" gate="G$1" x="-55.88" y="5.08"/>
 <instance part="R29" gate="G$1" x="-55.88" y="20.32" rot="R270"/>
 <instance part="-4.5V" gate="G$1" x="30.48" y="-7.62"/>
@@
 <instance part="SUPPLY39" gate="G$1" x="68.58" y="-38.1"/>
 <instance part="JP_POW" gate="B" x="-88.9" y="-33.02" rot="R90"/>
+<instance part="GND1" gate="1" x="-55.88" y="5.08"/>
+<instance part="GND2" gate="1" x="-25.4" y="5.08"/>
+<instance part="GND3" gate="1" x="27.94" y="5.08"/>
+<instance part="GND4" gate="1" x="40.64" y="5.08"/>
 </instances>
 <busses>
@@
 <pinref part="SJ_A/DGND2" gate="1" pin="1"/>
 <wire x1="78.74" y1="-10.16" x2="83.82" y2="-10.16" width="0.1524" layer="91"/>
-</segment>
-<segment>
-<pinref part="C33" gate="G$1" pin="1"/>
-<pinref part="SUPPLY37" gate="G$1" pin="AGND"/>
-<wire x1="40.64" y1="7.62" x2="40.64" y2="12.7" width="0.1524" layer="91"/>
 </segment>
 <segment>
@@
 <wire x1="30.48" y1="-66.04" x2="30.48" y2="-83.82" width="0.1524" layer="91"/>
 <pinref part="SUPPLY26" gate="G$1" pin="AGND"/>
-</segment>
-<segment>
-<pinref part="U11" gate="G$1" pin="LV"/>
-<wire x1="20.32" y1="33.02" x2="27.94" y2="33.02" width="0.1524" layer="91"/>
-<wire x1="27.94" y1="33.02" x2="27.94" y2="7.62" width="0.1524" layer="91"/>
-<pinref part="SUPPLY27" gate="G$1" pin="AGND"/>
-</segment>
-<segment>
-<pinref part="U11" gate="G$1" pin="GND"/>
-<wire x1="-15.24" y1="33.02" x2="-25.4" y2="33.02" width="0.1524" layer="91"/>
-<wire x1="-25.4" y1="33.02" x2="-25.4" y2="7.62" width="0.1524" layer="91"/>
-<pinref part="SUPPLY28" gate="G$1" pin="AGND"/>
-</segment>
-<segment>
-<pinref part="R29" gate="G$1" pin="2"/>
-<pinref part="SUPPLY30" gate="G$1" pin="AGND"/>
-<wire x1="-55.88" y1="15.24" x2="-55.88" y2="7.62" width="0.1524" layer="91"/>
 </segment>
 <segment>
@@
 </segment>
 </net>
+<net name="PGND" class="0">
+<segment>
+<pinref part="R29" gate="G$1" pin="2"/>
+<wire x1="-55.88" y1="15.24" x2="-55.88" y2="7.62" width="0.1524" layer="91"/>
+<pinref part="GND1" gate="1" pin="GND"/>
+</segment>
+<segment>
+<pinref part="U11" gate="G$1" pin="GND"/>
+<wire x1="-15.24" y1="33.02" x2="-25.4" y2="33.02" width="0.1524" layer="91"/>
+<wire x1="-25.4" y1="33.02" x2="-25.4" y2="7.62" width="0.1524" layer="91"/>
+<pinref part="GND2" gate="1" pin="GND"/>
+</segment>
+<segment>
+<pinref part="U11" gate="G$1" pin="LV"/>
+<wire x1="20.32" y1="33.02" x2="27.94" y2="33.02" width="0.1524" layer="91"/>
+<wire x1="27.94" y1="33.02" x2="27.94" y2="7.62" width="0.1524" layer="91"/>
+<pinref part="GND3" gate="1" pin="GND"/>
+</segment>
+<segment>
+<pinref part="C33" gate="G$1" pin="1"/>
+<wire x1="40.64" y1="7.62" x2="40.64" y2="12.7" width="0.1524" layer="91"/>
+<pinref part="GND4" gate="1" pin="GND"/>
+</segment>
+</net>

Commit message: More design for V2.0.
Parts:
- removed SJ_A/DGND1, SJ_A/DGND2: (no value), jumper:SJ
- added A_I/O1: PINHD-2X5/90, adafruit:PINHD-2X5/90
- U1, U17: value OPA4209AIPWMOD -> OPA4209
Connections:
- removed net N$8: BB1.GND@1, SJ_A/DGND1.1
- new net GPIO_0: A_I/O1.3, BB1.GPIO2_6
- new net GPIO_1: A_I/O1.4, BB1.GPIO2_7
- new net GPIO_2: A_I/O1.5, BB1.GPIO2_8
- new net GPIO_3: A_I/O1.6, BB1.GPIO2_9
- new net GPIO_4: A_I/O1.7, BB1.GPIO2_10
- new net GPIO_5: A_I/O1.8, BB1.GPIO2_11
- new net GPIO_6: A_I/O1.9, BB1.GPIO2_12
- new net GPIO_7: A_I/O1.10, BB1.GPIO2_13
- net AGND: no longer BB1.GND@2, SJ_A/DGND2.1
- net DGND: now also A_I/O1.1, A_I/O1.2, BB1.GND@1; no longer SJ_A/DGND1.2, SJ_A/DGND2.2
- net N$14: now also S1.4; no longer S1.3
- net N$18: now also S1.3; no longer S1.4
Other:
- note added: "Ground Link"
- moved on the sheet: A_I/O, S1

Commit message: Started laying out v2.0.
Parts:
- removed C43, C44, C45: 0.1uF, rcl:C-EUC0603
- removed C46, C47, C48: 1uF, rcl:C-EUC0603
- removed U11: LM2663, ti-extended:LM2663
- removed U12: MAX1735, Maxim_By_element14_Batch_1:MAX1735EUK25+T
- removed U13: TLV70245, ti-extended:TLV70025DDCR
- removed U16: 24C, on-semiconductor-01:24C
- removed U17: OPA4209, ti-extended:OPA4209AIPWMOD
- added C16: 1uF, rcl:C-EUC0603
- added C17, C18, C19, C8: 0.1uF, rcl:C-EUC0603
- added C20, C21, C22, C23: (no value), rcl:C-EUC0603
- added C7: 1nF, rcl:C-EUC0603
- added R21: 680, rcl:R-US_R0603
- added R22: 10k, rcl:R-US_R0603
- added U2: ADS8331, ti-extended:ADS8331IBPW
- added U3: AD5686, analog-devices-02:AD5686RARUZ
- added U4: OPA4209, ti-extended:OPA4209AIPWMOD
- added U6: TPS7A3001, ti-extended:TPS7A3001DGNR
- added U7: TPS7A4901, ti-extended:TPS7A4901DGNR
- -4.5V: value TPB1,27 -> TPPAD1-17; device testpad:TPB1,27 -> testpad:TPPAD1-17
- C1, C2: value 0.1uF -> 4.7uF; device rcl:C-EUC0603 -> rcl:C-EUC0805
- C10: value 4.7uF -> 1nF; device rcl:C-EUC0805 -> rcl:C-EUC0603
- C11: value 1nF -> 22uF
- C12: value 1nF -> 10uF; device rcl:C-EUC0603 -> rcl:C-USC0805
- C13, C14: value 1nF -> 0.1uF
- C15: value 22uF -> 1uF
- C24: value 0.1uF -> 10uF; device rcl:C-EUC0603 -> resistor:C-EUC1206
- C25: value (none) -> 10uF; device rcl:C-EUC0603 -> resistor:C-EUC1206
- C26: value 10uF -> 22uF; device rcl:C-USC0805 -> resistor:C-EUC1206
- C27, C28: value 0.1uF -> 10nF
- C29, C30: value (none) -> 10nF
- C3, C4: value 0.1uF -> 1nF
- C31: value (none) -> 22uF; device rcl:C-EUC0603 -> resistor:C-EUC1206
- C32, C33: value 47uF -> 10uF; device rcl:C-USC1206 -> resistor:C-EUC1206
- C34: value 10uF -> 1uF; device rcl:C-EUC0805 -> rcl:C-EUC0603
- C35, C37: value 1uF -> 0.1uF; device rcl:C-EUC0805 -> rcl:C-EUC0603
- C36: device rcl:C-EUC0805 -> rcl:C-EUC0603
- C38: value 4.7uF -> 1uF; device rcl:C-USC1206 -> rcl:C-EUC0603
- C39: value 1uF -> 4.7uF; device rcl:C-EUC0603 -> rcl:C-USC1206
- C40: value 1uF -> 0.1uF
- C9: value 4.7uF -> 0.1uF; device rcl:C-EUC0805 -> rcl:C-EUC0603
- R10: value 100 -> 680
- R11, R12: value 100 -> 340
- R13: value 100 -> 10
- R14: value 10 -> 10k
- R19: value 680 -> 10k
- R23: value (none) -> 680
- R24, R9: value 10k -> 680
- R29: value 10k -> (none)
- R30: value 100k -> 10k
- R31: value 261k -> 4.7k
- R32: value 2k -> 13.5k
- R33: value 2k -> 4.7k
- R34: value 10k -> 13.5k
- R35: value 10k -> 2k
- R36: value 10k -> 2k; device boneclamp:TRIM_US-M84W -> rcl:R-US_R0603
- R37: value 4.75k -> 10k; device rcl:R-US_R0603 -> boneclamp:TRIM_US-M84W
- R38, R39: value 4.75k -> 10k
- R40: value 10k -> 4.75k
- R41, R42: value 5.6k -> 4.75k
- R44, R45: value 680 -> 5.6k
- R5, R7: value 680 -> 100
- R6, R8: value 340 -> 100
- U10: value AD5686 -> 24C; device analog-devices-02:AD5686RARUZ -> on-semiconductor-01:24C
- U5: value ADS8331 -> LM2663; device ti-extended:ADS8331IBPW -> ti-extended:LM2663
- renumbered U14 to U8, U15 to U9
Connections:
- removed net N$5: R30.1, R31.1, U12.SET
- new net AGND1: C30.2, R33.2, R34.1, U7.FB
- new net AGND2: C29.2, R31.2, R32.1, U6.FB
- new net N$1: C28.1, U7.NR/SS
- new net N$2: C27.1, U6.NR/SS
- net +4.5V: now also C12.1, C13.1, C15.1, C17.1, C2.2, C30.1, C33.1, C34.1, C35.1, C36.2, C5.1, C8.1, R33.1, R35.2, U2.VA, U3.VDD, U4.V+, U7.OUT; no longer C1.1, C10.2, C26.1, C27.1, C37.1, C39.2, C4.1, C41.1, C46.1, C48.1, C6.1, R32.2, U10.VDD, U13.OUT, U17.V+, U5.VA
- net -4.5V: now also C16.1, C18.1, C29.1, C32.1, C34.2, C6.1, C9.1, R31.1, U4.V-, U6.OUT; no longer C2.1, C3.1, C35.1, C46.2, C47.1, C5.1, R31.2, U12.OUT, U17.V-
- net ADC_-IN_A: now also R2.1, R4.2, U1.-IN_A; no longer R1.1, R3.2, U17.-IN_A
- net ADC_-IN_B: now also R1.1, R3.2, U1.-IN_B; no longer R2.1, R4.2, U17.-IN_B
- net ADC_-IN_C: now also R11.2, R9.1, U1.-IN_C; no longer R5.1, R6.2, U17.-IN_C
- net ADC_-IN_D: now also R10.1, R12.2, U1.-IN_D; no longer R7.1, R8.2, U17.-IN_D
- net ADC_A: now also R2.2; no longer R1.2
- net ADC_A+: now also R4.1, R5.2, U1.OUT_A; no longer R10.2, R3.1, U17.OUT_A
- net ADC_B: now also R1.2; no longer R2.2
- net ADC_B+: now also R3.1, R6.2, U1.OUT_B; no longer R11.2, R4.1, U17.OUT_B
- net ADC_C: now also R9.2; no longer R5.2
- net ADC_C+: now also R11.1, R7.2, U1.OUT_C; no longer R12.2, R6.1, U17.OUT_C
- net ADC_D: now also R10.2; no longer R7.2
- net ADC_D+: now also R12.1, R8.2, U1.OUT_D; no longer R13.2, R8.1, U17.OUT_D
- net AGND: now also C12.2, C13.2, C15.2, C16.2, C17.2, C18.2, C19.2, C2.1, C20.2, C21.2, C22.2, C23.2, C28.2, C3.1, C32.2, C33.2, C36.1, C38.1, C39.2, C4.1, C40.2, C7.1, C8.2, R29.1, R32.2, R34.2, R37.A, U2.AGND, U2.COM, U2.DGND, U2.REF-, U3.GND, U6.EP, U6.GND, U7.EP, U7.GND; no longer C12.1, C13.1, C14.1, C15.1, C2.2, C26.2, C29.2, C3.2, C30.2, C31.2, C34.2, C36.2, C38.2, C39.1, C4.2, C40.1, C42.2, C43.2, C44.2, C47.2, C48.2, R23.1, R30.2, R36.A, U10.GND, U12.GND, U13.GND, U5.AGND, U5.COM, U5.DGND, U5.REF-
- net DAC_+IN_A: now also U4.+IN_A; no longer U1.+IN_A
- net DAC_+IN_B: now also U4.+IN_B; no longer U1.+IN_B
- net DAC_+IN_C: now also U4.+IN_C; no longer U1.+IN_C
- net DAC_+IN_D: now also U4.+IN_D; no longer U1.+IN_D
- net DAC_-IN_A: now also R15.1, R17.2, U4.-IN_A; no longer R44.1, R45.2, U1.-IN_A
- net DAC_-IN_B: now also R16.1, R18.2, U4.-IN_B; no longer R15.1, R16.2, U1.-IN_B
- net DAC_-IN_C: now also R20.1, R23.2, U4.-IN_C; no longer R17.1, R18.2, U1.-IN_C
- net DAC_-IN_D: now also R21.1, R24.2, U4.-IN_D; no longer R19.1, R20.2, U1.-IN_D
- net DAC_A: now also R17.1, U4.OUT_A; no longer R45.1, U1.OUT_A
- net DAC_A+: now also C23.1, R29.2, U3.VOUTA; no longer C31.1, R28.2, U10.VOUTA
- net DAC_B: now also R18.1, U4.OUT_B; no longer R16.1, U1.OUT_B
- net DAC_B+: now also C22.1, R28.2, U3.VOUTB; no longer C30.1, R27.2, U10.VOUTB
- net DAC_C: now also R23.1, U4.OUT_C; no longer R18.1, U1.OUT_C
- net DAC_C+: now also C21.1, R27.2, U3.VOUTC; no longer C29.1, R26.2, U10.VOUTC
- net DAC_D: now also R24.1, U4.OUT_D; no longer R20.1, U1.OUT_D
- net DAC_D+: now also C20.1, R26.2, U3.VOUTD; no longer C25.1, R23.2, U10.VOUTD
- net DAC_LDAC: now also R22.1, U3.LDAC*; no longer R25.1, U10.LDAC*
- net DGND: now also C14.2, C42.2, U10.GND, U3.GAIN; no longer C28.2, C45.2, U10.GAIN, U16.GND
- net I2C2_SCL: now also R44.1, U10.SCL; no longer R41.1, U16.SCL
- net I2C2_SDA: now also R45.1, U10.SDA; no longer R42.1, U16.SDA
- net N$11: now also R25.1, U3.RSTSEL; no longer R43.1, U10.RSTSEL
- net N$14: now also R40.1, U10.A0; no longer R37.1, U16.A0
- net N$16: now also C11.2, R13.1, U2.REF+; no longer C15.2, R14.1, U5.REF+
- net N$18: now also R41.1, U10.A1; no longer R38.1, U16.A1
- net N$19: now also R42.1, U10.A2; no longer R39.1, U16.A2
- net N$20: now also R35.1; no longer R32.1
- net N$22: now also R43.1, U10.WP; no longer R40.1, U16.WP
- net N$24: now also U2.ADCIN, U2.MUXOUT; no longer U5.ADCIN, U5.MUXOUT
- net N$32: now also C38.2; no longer C40.2
- net N$33: now also C26.1, U5.CAP+; no longer C32.1, U11.CAP+
- net N$34: now also C26.2, U5.CAP-; no longer C32.2, U11.CAP-
- net N$4: now also C37.1, R37.S; no longer C44.1, R36.S
- net N$40: now also C3.2, R5.1, U2.IN0; no longer C11.2, R10.1, U5.IN0
- net N$41: now also C4.2, R6.1, U2.IN1; no longer C12.2, R11.1, U5.IN1
- net N$42: now also C7.2, R7.1, U2.IN2; no longer C13.2, R12.1, U5.IN2
- net N$43: now also C10.2, R8.1, U2.IN3; no longer C14.2, R13.1, U5.IN3
- net N$7: now also R36.1; no longer R33.1
- net N$9: now also R39.2; no longer R35.2
- net PGND: now also C31.1, R30.2, U5.GND, U5.LV; no longer C33.1, R29.2, U11.GND, U11.LV
- net SPI0: now also U2.FS/~CS; no longer U5.FS/~CS
- net SPI1: now also U3.SYNC*; no longer U10.SYNC*
- net SPI2: now also U2.SCLK, U3.SCLK; no longer U10.SCLK, U5.SCLK
- net SPI3: now also U2.SDI, U3.SDIN; no longer U10.SDIN, U5.SDI
- net SPI4: now also U2.SDO, U3.SDO; no longer U10.SDO, U5.SDO
- net SPI5: now also U2.~CONVST; no longer U5.~CONVST
- net VBIAS: now also C41.1, R39.1, U1.+IN_A, U1.+IN_B, U1.+IN_C, U1.+IN_D; no longer C43.1, R35.1, U17.+IN_A, U17.+IN_B, U17.+IN_C, U17.+IN_D
- net VDD_5V: now also U5.V+; no longer U11.V+
- net VDD_COM: now also C25.1, U7.EN, U7.IN; no longer C36.1, U13.EN, U13.IN
- net VDD_EXT: now also R30.1, R36.2, U5.SD; no longer R29.1, R33.2, U11.SD
- net VDRIVE: now also C1.1, C14.1, C42.1, R14.2, R19.2, R22.2, R44.2, R45.2, U10.VCC, U2.VBD, U3.VDRIVE; no longer C28.1, C45.1, C9.1, R24.2, R37.2, R38.2, R39.2, R9.2, U10.VDRIVE, U16.VCC, U5.VBD
- net VREF: now also C19.1, C40.1, R13.2, R16.2, R20.2, R21.2, R38.1, U3.VREF; no longer C24.1, C42.1, R14.2, R17.2, R19.2, R34.1, R44.2, U10.VREF
- net VREF_NOFILT: now also R37.E, R38.2; no longer R34.2, R36.E
- net VREF_PRE: now also C39.1; no longer C38.1
- net VSS_COM: now also C24.1, U6.EN, U6.IN; no longer C34.1, U12.IN, U12.~SHDN
- net VSS_PRE: now also C31.2, U5.VOUT; no longer C33.2, U11.VOUT
- net ~RST: now also R14.1, R19.1, U2.~RESET, U3.RESET*; no longer R24.1, R9.1, U10.RESET*, U5.~RESET
Other:
- note removed: "Vout = -1.25*(1 + R1/R2) = -4.5V"
