File: bob/bnc-bob/bnc_BOB.sch (EAGLE design)
At the start: 9 parts

Commit message: Finished CMOS to TTL BOB. Cleaned up directory structure.
Parts:
- AI_B, AI_C, AI_D, AO_A, AO_B, AO_C, AO_D: device con-coax:BN35N61 -> puggleboard:BN35N61
- A_I/O: value PINHD-2X5 -> PINHD-2X5-IDC-SMD; device adafruit:PINHD-2X5 -> puggleboard:PINHD-2X5-IDC-SMD
Other:
- moved on the sheet: A_I/O
Changed lines of the file:
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@@
 <layer number="97" name="Info" color="7" fill="1" visible="yes" active="yes"/>
 <layer number="98" name="Guide" color="6" fill="1" visible="yes" active="yes"/>
+<layer number="99" name="SpiceOrder" color="5" fill="1" visible="yes" active="yes"/>
 <layer number="100" name="Muster" color="7" fill="1" visible="no" active="no"/>
 <layer number="101" name="Patch_Top" color="12" fill="4" visible="yes" active="yes"/>
@@
 </classes>
 <parts>
-<part name="A_I/O" library="adafruit" deviceset="PINHD-2X5" device="" value="PINHD-2X5"/>
+<part name="A_I/O" library="puggleboard" deviceset="PINHD-2X5" device="-IDC-SMD" value="PINHD-2X5-IDC-SMD"/>
 <part name="AI_A" library="con-coax" deviceset="BN35N61" device="" value="5-1634503-1"/>
-<part name="AI_B" library="con-coax" deviceset="BN35N61" device="" value="5-1634503-1"/>
-<part name="AI_C" library="con-coax" deviceset="BN35N61" device="" value="5-1634503-1"/>
-<part name="AI_D" library="con-coax" deviceset="BN35N61" device="" value="5-1634503-1"/>
-<part name="AO_A" library="con-coax" deviceset="BN35N61" device="" value="5-1634503-1"/>
-<part name="AO_B" library="con-coax" deviceset="BN35N61" device="" value="5-1634503-1"/>
-<part name="AO_C" library="con-coax" deviceset="BN35N61" device="" value="5-1634503-1"/>
-<part name="AO_D" library="con-coax" deviceset="BN35N61" device="" value="5-1634503-1"/>
+<part name="AI_B" library="puggleboard" deviceset="BN35N61" device="" value="5-1634503-1"/>
+<part name="AI_C" library="puggleboard" deviceset="BN35N61" device="" value="5-1634503-1"/>
+<part name="AI_D" library="puggleboard" deviceset="BN35N61" device="" value="5-1634503-1"/>
+<part name="AO_A" library="puggleboard" deviceset="BN35N61" device="" value="5-1634503-1"/>
+<part name="AO_B" library="puggleboard" deviceset="BN35N61" device="" value="5-1634503-1"/>
+<part name="AO_C" library="puggleboard" deviceset="BN35N61" device="" value="5-1634503-1"/>
+<part name="AO_D" library="puggleboard" deviceset="BN35N61" device="" value="5-1634503-1"/>
 <part name="SUPPLY1" library="supply2" deviceset="AGND" device=""/>
 <part name="SUPPLY2" library="supply2" deviceset="AGND" device=""/>

Commit message: Finished BOMs (and integrated parts into database) for all the BOBs. Now must do for the main board. Will take a while.
Parts:
- AI_A: device con-coax:BN35N61 -> puggleboard:BN35N61
Changed lines of the file:
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@@
 <parts>
 <part name="A_I/O" library="puggleboard" deviceset="PINHD-2X5" device="-IDC-SMD" value="PINHD-2X5-IDC-SMD"/>
-<part name="AI_A" library="con-coax" deviceset="BN35N61" device="" value="5-1634503-1"/>
+<part name="AI_A" library="puggleboard" deviceset="BN35N61" device="" value="5-1634503-1"/>
 <part name="AI_B" library="puggleboard" deviceset="BN35N61" device="" value="5-1634503-1"/>
 <part name="AI_C" library="puggleboard" deviceset="BN35N61" device="" value="5-1634503-1"/>
