File: bob/ttl-bob/ttl-bob.sch (EAGLE design)
At the start: 9 parts, among them U1 TXB0108

Commit message: Finished BOMs (and integrated parts into database) for all the BOBs. Now must do for the main board. Will take a while.
Parts:
- ON: value LEDGREEN-CHIP0805 -> LEDGREEN_0805; device puggleboard:LEDGREEN-CHIP0805 -> puggleboard:LEDGREEN_0805
Changed lines of the file:
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@@
 <part name="C1" library="puggleboard" deviceset="C" device="_0805" value="10uF"/>
 <part name="GND22" library="supply1" deviceset="GND" device=""/>
-<part name="ON" library="puggleboard" deviceset="LED" device="-CHIP0805" technology="GREEN" value="LEDGREEN-CHIP0805"/>
+<part name="ON" library="puggleboard" deviceset="LED" device="_0805" technology="GREEN" value="LEDGREEN_0805"/>
 <part name="R1" library="puggleboard" deviceset="R" device="_0603" value="1k">
 <attribute name="DK" value="P1.00KHCT-ND"/>
